Commit message: feat(sim): split leg into 3 articulated mesh segments

File: code/simulation/facehugger.urdf (robot description, URDF)
Before this commit: robot facehugger, 17 links, 16 joints
Links:
- removed link fl_foot
- removed link fr_foot
- removed link rl_foot
- removed link rr_foot
- link fl_lower_leg: geometry collision box size=0.020 0.020 0.0774; collision sphere radius=0.008
- link fl_shoulder: geometry collision box size=0.080 0.025 0.025; visual mesh filename=meshes/leg_shoulder.stl scale=0.001 0.001 0.001
- link fl_upper_leg: geometry collision box size=0.025 0.025 0.075; visual mesh filename=meshes/leg_upper.stl scale=0.001 0.001 0.001
- link fr_lower_leg: geometry collision box size=0.020 0.020 0.0774; collision sphere radius=0.008
- link fr_shoulder: geometry collision box size=0.080 0.025 0.025; visual mesh filename=meshes/leg_shoulder.stl scale=0.001 0.001 0.001
- link fr_upper_leg: geometry collision box size=0.025 0.025 0.075; visual mesh filename=meshes/leg_upper.stl scale=0.001 0.001 0.001
- link rl_lower_leg: geometry collision box size=0.020 0.020 0.0774; collision sphere radius=0.008
- link rl_shoulder: geometry collision box size=0.080 0.025 0.025; visual mesh filename=meshes/leg_shoulder.stl scale=0.001 0.001 0.001
- link rl_upper_leg: geometry collision box size=0.025 0.025 0.075; visual mesh filename=meshes/leg_upper.stl scale=0.001 0.001 0.001
- link rr_lower_leg: geometry collision box size=0.020 0.020 0.0774; collision sphere radius=0.008
- link rr_shoulder: geometry collision box size=0.080 0.025 0.025; visual mesh filename=meshes/leg_shoulder.stl scale=0.001 0.001 0.001
- link rr_upper_leg: geometry collision box size=0.025 0.025 0.075; visual mesh filename=meshes/leg_upper.stl scale=0.001 0.001 0.001
Joints:
- removed joint fl_foot_joint
- removed joint fr_foot_joint
- removed joint rl_foot_joint
- removed joint rr_foot_joint

Commit message: feat(simulation): add Fusion→URDF pipeline with real geometry and inertia
- ExportBodiesToURDF.py: recursive Fusion assembly traversal, outputs
  fusion_export.json + STLs to code/simulation/ via repo-relative path;
  collects physical properties (mass, CoM, inertia) from Fusion API
- facehugger_config.yaml: robot hierarchy config mapping Fusion construction
  geometry to URDF links/joints; 4-leg instantiation from one template
- generate_urdf.py: reads export JSON + config, generates facehugger.urdf
  with precise joint origins, axes, and inertial data from Fusion
- facehugger.urdf: regenerated with real coordinates from Fusion geometry,
  correct DS3230MG effort (2.94 Nm), 4 independent leg chains (12 joints)
- exported_meshes/: STLs exported directly from Fusion assembly
- requirements.txt: pybullet + pyyaml, with conda-forge install note for macOS

File: code/simulation/facehugger.urdf (robot description, URDF)
Before this commit: robot facehugger, 13 links, 12 joints
Links:
- removed link body
- removed link fl_lower_leg
- removed link fl_shoulder
- removed link fl_upper_leg
- removed link fr_lower_leg
- removed link fr_shoulder
- removed link fr_upper_leg
- removed link rl_lower_leg
- removed link rl_shoulder
- removed link rl_upper_leg
- removed link rr_lower_leg
- removed link rr_shoulder
- removed link rr_upper_leg
- added link base_link, mass 0.741395; collision mesh filename=meshes/QuadrupedBody.stl scale=0.001 0.001 0.001; visual mesh filename=meshes/QuadrupedBody.stl scale=0.001 0.001 0.001
- added link bl_link1, mass 0.144017; collision mesh filename=meshes/leg_shoulder.stl scale=0.001 0.001 0.001; visual mesh filename=meshes/leg_shoulder.stl scale=0.001 0.001 0.001
- added link bl_link2, mass 0.173381; collision mesh filename=meshes/leg_upper.stl scale=0.001 0.001 0.001; visual mesh filename=meshes/leg_upper.stl scale=0.001 0.001 0.001
- added link bl_link3, mass 0.111653; collision mesh filename=meshes/leg_lower.stl scale=0.001 0.001 0.001; visual mesh filename=meshes/leg_lower.stl scale=0.001 0.001 0.001
- added link br_link1, mass 0.144017; collision mesh filename=meshes/leg_shoulder.stl scale=0.001 0.001 0.001; visual mesh filename=meshes/leg_shoulder.stl scale=0.001 0.001 0.001
- added link br_link2, mass 0.173381; collision mesh filename=meshes/leg_upper.stl scale=0.001 0.001 0.001; visual mesh filename=meshes/leg_upper.stl scale=0.001 0.001 0.001
- added link br_link3, mass 0.111653; collision mesh filename=meshes/leg_lower.stl scale=0.001 0.001 0.001; visual mesh filename=meshes/leg_lower.stl scale=0.001 0.001 0.001
- added link fl_link1, mass 0.144017; collision mesh filename=meshes/leg_shoulder.stl scale=0.001 0.001 0.001; visual mesh filename=meshes/leg_shoulder.stl scale=0.001 0.001 0.001
- added link fl_link2, mass 0.173381; collision mesh filename=meshes/leg_upper.stl scale=0.001 0.001 0.001; visual mesh filename=meshes/leg_upper.stl scale=0.001 0.001 0.001
- added link fl_link3, mass 0.111653; collision mesh filename=meshes/leg_lower.stl scale=0.001 0.001 0.001; visual mesh filename=meshes/leg_lower.stl scale=0.001 0.001 0.001
- added link fr_link1, mass 0.144017; collision mesh filename=meshes/leg_shoulder.stl scale=0.001 0.001 0.001; visual mesh filename=meshes/leg_shoulder.stl scale=0.001 0.001 0.001
- added link fr_link2, mass 0.173381; collision mesh filename=meshes/leg_upper.stl scale=0.001 0.001 0.001; visual mesh filename=meshes/leg_upper.stl scale=0.001 0.001 0.001
- added link fr_link3, mass 0.111653; collision mesh filename=meshes/leg_lower.stl scale=0.001 0.001 0.001; visual mesh filename=meshes/leg_lower.stl scale=0.001 0.001 0.001
Joints:
- removed joint rl_hip_joint
- removed joint rl_knee_joint
- removed joint rl_shoulder_joint
- removed joint rr_hip_joint
- removed joint rr_knee_joint
- removed joint rr_shoulder_joint
- added joint bl_hip_joint: type revolute, parent bl_link1, child bl_link2, origin xyz=0.022595 0.050920 0.010446 rpy=0 0 0.0, axis 1.0 0.0 -0.0, limit lower=-1.570796 upper=1.570796 effort=2.94 velocity=5.0
- added joint bl_knee_joint: type revolute, parent bl_link2, child bl_link3, origin xyz=0.000005 0.094700 0.000000 rpy=0 0 0.0, axis 1.0 0.0 -0.0, limit lower=-2.356194 upper=0.523599 effort=2.94 velocity=5.0
- added joint bl_shoulder_joint: type revolute, parent base_link, child bl_link1, origin xyz=-0.055401 -0.046222 -0.009000 rpy=0 0 0.0, axis 0.0 0.0 1.0, limit lower=-1.570796 upper=1.570796 effort=2.94 velocity=5.0
- added joint br_hip_joint: type revolute, parent br_link1, child br_link2, origin xyz=0.022595 0.050920 0.010446 rpy=0 0 0.0, axis 1.0 0.0 -0.0, limit lower=-1.570796 upper=1.570796 effort=2.94 velocity=5.0
- added joint br_knee_joint: type revolute, parent br_link2, child br_link3, origin xyz=0.000005 0.094700 0.000000 rpy=0 0 0.0, axis 1.0 0.0 -0.0, limit lower=-2.356194 upper=0.523599 effort=2.94 velocity=5.0
- added joint br_shoulder_joint: type revolute, parent base_link, child br_link1, origin xyz=0.055401 -0.046222 -0.009000 rpy=0 0 3.141593, axis 0.0 0.0 1.0, limit lower=-1.570796 upper=1.570796 effort=2.94 velocity=5.0
- joint fl_hip_joint: axis 0 1 0 -> 1.0 0.0 -0.0; child fl_upper_leg -> fl_link2; limit lower=-1.5708 upper=1.5708 effort=1.47 velocity=5.0 -> lower=-1.570796 upper=1.570796 effort=2.94 velocity=5.0; origin xyz=-0.08 0 0 rpy=0 0 0 -> xyz=0.022595 0.050920 0.010446 rpy=0 0 0.0; parent fl_shoulder -> fl_link1
- joint fl_knee_joint: axis 0 1 0 -> 1.0 0.0 -0.0; child fl_lower_leg -> fl_link3; limit lower=-2.356 upper=0.5 effort=1.47 velocity=5.0 -> lower=-2.356194 upper=0.523599 effort=2.94 velocity=5.0; origin xyz=0 0 -0.075 rpy=0 0 0 -> xyz=0.000005 0.094700 0.000000 rpy=0 0 0.0; parent fl_upper_leg -> fl_link2
- joint fl_shoulder_joint: axis 0 0 1 -> 0.0 0.0 1.0; child fl_shoulder -> fl_link1; limit lower=-2.356 upper=2.356 effort=1.47 velocity=5.0 -> lower=-1.570796 upper=1.570796 effort=2.94 velocity=5.0; origin xyz=-0.080 0.105 0.025 rpy=0 0 0 -> xyz=-0.055401 0.046222 -0.009000 rpy=0 0 3.141593; parent body -> base_link
- joint fr_hip_joint: axis 0 1 0 -> 1.0 0.0 -0.0; child fr_upper_leg -> fr_link2; limit lower=-1.5708 upper=1.5708 effort=1.47 velocity=5.0 -> lower=-1.570796 upper=1.570796 effort=2.94 velocity=5.0; origin xyz=-0.08 0 0 rpy=0 0 0 -> xyz=0.022595 0.050920 0.010446 rpy=0 0 0.0; parent fr_shoulder -> fr_link1
- joint fr_knee_joint: axis 0 1 0 -> 1.0 0.0 -0.0; child fr_lower_leg -> fr_link3; limit lower=-2.356 upper=0.5 effort=1.47 velocity=5.0 -> lower=-2.356194 upper=0.523599 effort=2.94 velocity=5.0; origin xyz=0 0 -0.075 rpy=0 0 0 -> xyz=0.000005 0.094700 0.000000 rpy=0 0 0.0; parent fr_upper_leg -> fr_link2
- joint fr_shoulder_joint: axis 0 0 1 -> 0.0 0.0 1.0; child fr_shoulder -> fr_link1; limit lower=-2.356 upper=2.356 effort=1.47 velocity=5.0 -> lower=-1.570796 upper=1.570796 effort=2.94 velocity=5.0; origin xyz=0.080 0.105 0.025 rpy=0 0 3.14159 -> xyz=0.055401 0.046222 -0.009000 rpy=0 0 0.0; parent body -> base_link

Commit message: swap body mesh to FlexibleSkeletonWithMotorMounts

File: code/simulation/facehugger.urdf (robot description, URDF)
Before this commit: robot facehugger, 13 links, 12 joints
Links:
- link body: geometry collision box size=0.130 0.128 0.054; visual mesh filename=meshes/FlexibleSkeletonWithMotorMounts.stl scale=0.001 0.001 0.001
Joints:
- joint fl_shoulder_joint: origin xyz=-0.080 0.105 0.025 rpy=0 0 0 -> xyz=-0.040 0.050 0.025 rpy=0 0 0
- joint fr_shoulder_joint: origin xyz=0.080 0.105 0.025 rpy=0 0 3.14159 -> xyz=0.040 0.050 0.025 rpy=0 0 3.14159
- joint rl_shoulder_joint: origin xyz=-0.080 -0.105 0.025 rpy=0 0 0 -> xyz=-0.040 -0.050 0.025 rpy=0 0 0
- joint rr_shoulder_joint: origin xyz=0.080 -0.105 0.025 rpy=0 0 3.14159 -> xyz=0.040 -0.050 0.025 rpy=0 0 3.14159
