Commit message: chore(simulation): regenerate Fusion export + STLs + URDF
Regenerated outputs from the new rule-based Fusion exporter and
manifest-driven URDF generator.

- exported_meshes/QuadrupedBody.stl: now built via the `combined` rule;
  5 explicit parts (QuadrupedBody body + 4 LegMountXX bodies) transformed
  into world frame and concatenated. No electronics bodies baked in.
  Verified via animation/scripts/inspect_stl.py: 1 connected component,
  bbox x±65 / y±64 / z[-13,+41] mm.
- exported_meshes/leg_shoulder.stl, leg_upper.stl, leg_lower.stl:
  pre-re-origined so each link mesh's local (0,0,0) coincides with its
  URDF joint landmark (BodyToLink1Point / Link1ToLink2Point /
  Link2ToLink3Point). Lets the URDF emit <visual><origin xyz="0 0 0"/>.
- exported_meshes/servo.stl: new. ServoBase body only; reused at all
  twelve servo locations (3 per leg × 4 legs) in the URDF.
- fusion_export.json: gains `mesh_files` manifest describing each STL
  (source_type, source_occurrences, origin_shift_mm, parts,
  _servo_role_assignment). 19k+ lines due to the full occurrence tree
  including all electronics (still useful metadata for downstream tools).
- fusion_export.txt: corresponding human-readable tree.
- facehugger.urdf: 13 links × 25 visuals including 4 shoulder + 4 hip +
  4 knee servo meshes on their respective host links.

Co-Authored-By: Claude Opus 4.7 (1M context) <noreply@anthropic.com>

File: code/simulation/facehugger.urdf (robot description, URDF)
Before this commit: robot facehugger, 13 links, 12 joints
Links:
- link base_link: geometry collision mesh filename=exported_meshes/QuadrupedBody.stl scale=0.001 0.001 0.001; visual mesh filename=exported_meshes/QuadrupedBody.stl scale=0.001 0.001 0.001
- link bl_link1: geometry collision mesh filename=exported_meshes/leg_shoulder.stl scale=0.001 0.001 0.001; visual mesh filename=exported_meshes/leg_shoulder.stl scale=0.001 0.001 0.001
- link bl_link2: geometry collision mesh filename=exported_meshes/leg_upper.stl scale=0.001 0.001 0.001; visual mesh filename=exported_meshes/leg_upper.stl scale=0.001 0.001 0.001
- link bl_link3: geometry collision mesh filename=exported_meshes/leg_lower.stl scale=0.001 0.001 0.001; visual mesh filename=exported_meshes/leg_lower.stl scale=0.001 0.001 0.001
- link br_link1: geometry collision mesh filename=exported_meshes/leg_shoulder.stl scale=0.001 0.001 0.001; visual mesh filename=exported_meshes/leg_shoulder.stl scale=0.001 0.001 0.001
- link br_link2: geometry collision mesh filename=exported_meshes/leg_upper.stl scale=0.001 0.001 0.001; visual mesh filename=exported_meshes/leg_upper.stl scale=0.001 0.001 0.001
- link br_link3: geometry collision mesh filename=exported_meshes/leg_lower.stl scale=0.001 0.001 0.001; visual mesh filename=exported_meshes/leg_lower.stl scale=0.001 0.001 0.001
- link fl_link1: geometry collision mesh filename=exported_meshes/leg_shoulder.stl scale=0.001 0.001 0.001; visual mesh filename=exported_meshes/leg_shoulder.stl scale=0.001 0.001 0.001
- link fl_link2: geometry collision mesh filename=exported_meshes/leg_upper.stl scale=0.001 0.001 0.001; visual mesh filename=exported_meshes/leg_upper.stl scale=0.001 0.001 0.001
- link fl_link3: geometry collision mesh filename=exported_meshes/leg_lower.stl scale=0.001 0.001 0.001; visual mesh filename=exported_meshes/leg_lower.stl scale=0.001 0.001 0.001
- link fr_link1: geometry collision mesh filename=exported_meshes/leg_shoulder.stl scale=0.001 0.001 0.001; visual mesh filename=exported_meshes/leg_shoulder.stl scale=0.001 0.001 0.001
- link fr_link2: geometry collision mesh filename=exported_meshes/leg_upper.stl scale=0.001 0.001 0.001; visual mesh filename=exported_meshes/leg_upper.stl scale=0.001 0.001 0.001
- link fr_link3: geometry collision mesh filename=exported_meshes/leg_lower.stl scale=0.001 0.001 0.001; visual mesh filename=exported_meshes/leg_lower.stl scale=0.001 0.001 0.001
Joints:
- joint bl_hip_joint: origin xyz=0.022595 0.050920 0.010446 rpy=0 0 0.0 -> xyz=0.022595 0.050920 0.014446 rpy=0 0 0.0
- joint bl_shoulder_joint: limit lower=-1.570796 upper=1.570796 effort=2.94 velocity=5.0 -> lower=-3.141593 upper=3.141593 effort=2.94 velocity=5.0; origin xyz=-0.055401 -0.046222 -0.009000 rpy=0 0 0.0 -> xyz=-0.055401 -0.046222 -0.009000 rpy=0 0 1.570796
- joint br_hip_joint: origin xyz=0.022595 0.050920 0.010446 rpy=0 0 0.0 -> xyz=0.022595 0.050920 0.014446 rpy=0 0 0.0
- joint br_shoulder_joint: limit lower=-1.570796 upper=1.570796 effort=2.94 velocity=5.0 -> lower=-3.141593 upper=3.141593 effort=2.94 velocity=5.0; origin xyz=0.055401 -0.046222 -0.009000 rpy=0 0 3.141593 -> xyz=0.055401 -0.046222 -0.009000 rpy=0 0 1.570796
- joint fl_hip_joint: origin xyz=0.022595 0.050920 0.010446 rpy=0 0 0.0 -> xyz=0.022595 0.050920 0.014446 rpy=0 0 0.0
- joint fl_shoulder_joint: limit lower=-1.570796 upper=1.570796 effort=2.94 velocity=5.0 -> lower=-3.141593 upper=3.141593 effort=2.94 velocity=5.0; origin xyz=-0.055401 0.046222 -0.009000 rpy=0 0 3.141593 -> xyz=-0.055401 0.046222 -0.009000 rpy=0 0 1.570796
- joint fr_hip_joint: origin xyz=0.022595 0.050920 0.010446 rpy=0 0 0.0 -> xyz=0.022595 0.050920 0.014446 rpy=0 0 0.0
- joint fr_shoulder_joint: limit lower=-1.570796 upper=1.570796 effort=2.94 velocity=5.0 -> lower=-3.141593 upper=3.141593 effort=2.94 velocity=5.0; origin xyz=0.055401 0.046222 -0.009000 rpy=0 0 0.0 -> xyz=0.055401 0.046222 -0.009000 rpy=0 0 1.570796

Commit message: chore(simulation): regenerate URDF, servo STL, and Fusion export
Outputs rebuilt after:
- Re-origining servo.stl to ServoMountPoint (fusion_export.json's
  mesh_files.servo.stl gains origin_landmark="ServoMountPoint" and
  nonzero origin_shift_mm).
- Per-leg shoulder limits + simplified servo placements in the URDF.

URDF has 4 shoulder-servo visuals on base_link at the LegMountXX world
positions (rpy=0, xyz=LegMountXX); each leg's link2/link3 gain a
visual at xyz=(0,0,0). Per-leg shoulder joint limits in
[neutral ± 90°] form.

Co-Authored-By: Claude Opus 4.7 (1M context) <noreply@anthropic.com>

File: code/simulation/facehugger.urdf (robot description, URDF)
Before this commit: robot facehugger, 13 links, 12 joints
Joints:
- joint bl_shoulder_joint: limit lower=-3.141593 upper=3.141593 effort=2.94 velocity=5.0 -> lower=-3.926991 upper=-0.785398 effort=2.94 velocity=5.0; origin xyz=-0.055401 -0.046222 -0.009000 rpy=0 0 1.570796 -> xyz=-0.055401 -0.046222 -0.009000 rpy=0 0 -1.570796
- joint br_shoulder_joint: limit lower=-3.141593 upper=3.141593 effort=2.94 velocity=5.0 -> lower=-2.356194 upper=0.785398 effort=2.94 velocity=5.0; origin xyz=0.055401 -0.046222 -0.009000 rpy=0 0 1.570796 -> xyz=0.055401 -0.046222 -0.009000 rpy=0 0 -1.570796
- joint fl_shoulder_joint: limit lower=-3.141593 upper=3.141593 effort=2.94 velocity=5.0 -> lower=0.785398 upper=3.926991 effort=2.94 velocity=5.0; origin xyz=-0.055401 0.046222 -0.009000 rpy=0 0 1.570796 -> xyz=-0.055401 0.046222 -0.009000 rpy=0 0 -1.570796
- joint fr_shoulder_joint: limit lower=-3.141593 upper=3.141593 effort=2.94 velocity=5.0 -> lower=-0.785398 upper=2.356194 effort=2.94 velocity=5.0; origin xyz=0.055401 0.046222 -0.009000 rpy=0 0 1.570796 -> xyz=0.055401 0.046222 -0.009000 rpy=0 0 -1.570796

Commit message: feat(sim): Phase B — generate_urdf consumes CAD joints + per-side meshes + bracket visuals
generate_urdf.py + facehugger_config.yaml updated end-to-end against
PIPELINE_SPEC.md. The yaml is now the per-leg placement layer only;
joint kinematics come from fusion_export.json's `joints` array.

facehugger_config.yaml shape:
- base_link drops the `occurrences` documentation list (chassis is
  driven by ExportBodiesToURDF.EXPORT_RULES, not yaml).
- leg_template.joints is a thin mapping `cad_name → urdf_name +
  parent/child link`. axis_key / point_key / limits_deg removed —
  the generator pulls those from the CAD joint entry by name.
- leg_template.links.link1.mesh is now `"leg_shoulder_{side}.stl"`;
  generator substitutes {side} per leg. Link2 / Link3 stay shared.
- legs[] gets `side: L|R` (diagonal pair: {FL,BR}=L, {FR,BL}=R),
  `rpy_z_deg: 0|180` (back-of-pair flips 180° around its own
  LegMountPointXX), and `shoulder_limits_deg: [lower, upper]` per
  PIPELINE_SPEC §4 ([-105,+45] for -X-pointing FL/BL, [-45,+105]
  for +X-pointing FR/BR). shoulder_neutral_deg drops to 0 for all
  legs — zero is "leg pointing along chassis ±X".

generate_urdf.py changes:
- New `_primary_link_occurrence(mesh_entry)` pulls the link body's
  occurrence path from a mesh_files entry — combined-rule outputs
  are convention-of-first-part; body-rule outputs use
  source_occurrences[0]. Used for inertial physics lookup.
- Joint kinematics resolved from `export["joints"]` by name; raises
  if a required joint is missing from the array (use the JOINTS
  whitelist in the export script to add more).
- 4 new bracket visuals on base_link, one per leg: `leg_mount_L.stl`
  for FL/BR, `leg_mount_R.stl` for FR/BL. xyz = LegMountPointXX,
  rpy = (0,0,π) for back-of-pair (rotates the bracket geometry to
  face outward).
- 4 chassis-fixed shoulder-servo visuals on base_link kept.
- Free-standing hip/knee servo visuals on link2/link3 DROPPED — the
  hip servo body is rigidly part of leg_shoulder_{L,R}.stl per
  Link1RigidGroup, and the knee servo body is part of leg_lower.stl
  per Link3RigidGroup (combined-rule exports). Emitting them again
  would render the same geometry twice.
- Per-leg shoulder-joint <limit> uses shoulder_limits_deg directly;
  per-leg comment block reports side + rpy_z_deg + limits.

Verification on the latest export:
- 21 <visual> elements (chassis 1 + 4 brackets + 4 chassis shoulder
  servos + 4 link1 + 4 link2 + 4 link3, the link visuals double-
  counted via collision elements).
- 2× leg_shoulder_L.stl + 2× leg_shoulder_R.stl, 2× leg_mount_L.stl
  + 2× leg_mount_R.stl, 4× servo.stl on base_link only.
- Per-leg shoulder limits: FL [-105,+45], BR [-45,+105],
  FR [-45,+105], BL [-105,+45] in radians match PIPELINE_SPEC §4
  exactly. Hip/knee limits straight from CAD's Link2/Link3Revolute.

Cleanup riding along:
- legacy code/simulation/meshes/ folder (predecessor of
  exported_meshes/) deleted — stale content from a prior reorg.
- old code/simulation/exported_meshes/leg_shoulder.stl deleted
  (replaced by L/R variants).
- stray cad/scripts/fusion_export.txt deleted.

Co-Authored-By: Claude Opus 4.7 (1M context) <noreply@anthropic.com>

File: code/simulation/facehugger.urdf (robot description, URDF)
Before this commit: robot facehugger, 13 links, 12 joints
Links:
- link base_link: mass 0.741395 -> 0.631194; geometry collision mesh filename=exported_meshes/QuadrupedBody.stl scale=0.001 0.001 0.001; visual mesh filename=exported_meshes/QuadrupedBody.stl scale=0.001 0.001 0.001
- link bl_link1: geometry collision mesh filename=exported_meshes/leg_shoulder_R.stl scale=0.001 0.001 0.001; visual mesh filename=exported_meshes/leg_shoulder_R.stl scale=0.001 0.001 0.001
- link bl_link2: geometry collision mesh filename=exported_meshes/leg_upper.stl scale=0.001 0.001 0.001; visual mesh filename=exported_meshes/leg_upper.stl scale=0.001 0.001 0.001
- link bl_link3: geometry collision mesh filename=exported_meshes/leg_lower.stl scale=0.001 0.001 0.001; visual mesh filename=exported_meshes/leg_lower.stl scale=0.001 0.001 0.001
- link br_link1: geometry collision mesh filename=exported_meshes/leg_shoulder_L.stl scale=0.001 0.001 0.001; visual mesh filename=exported_meshes/leg_shoulder_L.stl scale=0.001 0.001 0.001
- link br_link2: geometry collision mesh filename=exported_meshes/leg_upper.stl scale=0.001 0.001 0.001; visual mesh filename=exported_meshes/leg_upper.stl scale=0.001 0.001 0.001
- link br_link3: geometry collision mesh filename=exported_meshes/leg_lower.stl scale=0.001 0.001 0.001; visual mesh filename=exported_meshes/leg_lower.stl scale=0.001 0.001 0.001
- link fl_link1: geometry collision mesh filename=exported_meshes/leg_shoulder_L.stl scale=0.001 0.001 0.001; visual mesh filename=exported_meshes/leg_shoulder_L.stl scale=0.001 0.001 0.001
- link fl_link2: geometry collision mesh filename=exported_meshes/leg_upper.stl scale=0.001 0.001 0.001; visual mesh filename=exported_meshes/leg_upper.stl scale=0.001 0.001 0.001
- link fl_link3: geometry collision mesh filename=exported_meshes/leg_lower.stl scale=0.001 0.001 0.001; visual mesh filename=exported_meshes/leg_lower.stl scale=0.001 0.001 0.001
- link fr_link1: geometry collision mesh filename=exported_meshes/leg_shoulder_R.stl scale=0.001 0.001 0.001; visual mesh filename=exported_meshes/leg_shoulder_R.stl scale=0.001 0.001 0.001
- link fr_link2: geometry collision mesh filename=exported_meshes/leg_upper.stl scale=0.001 0.001 0.001; visual mesh filename=exported_meshes/leg_upper.stl scale=0.001 0.001 0.001
- link fr_link3: geometry collision mesh filename=exported_meshes/leg_lower.stl scale=0.001 0.001 0.001; visual mesh filename=exported_meshes/leg_lower.stl scale=0.001 0.001 0.001
Joints:
- joint bl_hip_joint: axis 1.0 0.0 -0.0 -> 1.0 0.0 0.0; limit lower=-1.570796 upper=1.570796 effort=2.94 velocity=5.0 -> lower=-2.356194 upper=0.785398 effort=2.94 velocity=5.0
- joint bl_knee_joint: axis 1.0 0.0 -0.0 -> 1.0 0.0 0.0; limit lower=-2.356194 upper=0.523599 effort=2.94 velocity=5.0 -> lower=-1.570796 upper=1.570796 effort=2.94 velocity=5.0
- joint bl_shoulder_joint: limit lower=-3.926991 upper=-0.785398 effort=2.94 velocity=5.0 -> lower=-1.832596 upper=0.785398 effort=2.94 velocity=5.0; origin xyz=-0.055401 -0.046222 -0.009000 rpy=0 0 -1.570796 -> xyz=-0.041500 -0.049000 0.026000 rpy=0 0 3.141593
- joint br_hip_joint: axis 1.0 0.0 -0.0 -> 1.0 0.0 0.0; limit lower=-1.570796 upper=1.570796 effort=2.94 velocity=5.0 -> lower=-2.356194 upper=0.785398 effort=2.94 velocity=5.0
- joint br_knee_joint: axis 1.0 0.0 -0.0 -> 1.0 0.0 0.0; limit lower=-2.356194 upper=0.523599 effort=2.94 velocity=5.0 -> lower=-1.570796 upper=1.570796 effort=2.94 velocity=5.0
- joint br_shoulder_joint: limit lower=-2.356194 upper=0.785398 effort=2.94 velocity=5.0 -> lower=-0.785398 upper=1.832596 effort=2.94 velocity=5.0; origin xyz=0.055401 -0.046222 -0.009000 rpy=0 0 -1.570796 -> xyz=0.041500 -0.049000 0.026000 rpy=0 0 3.141593
- joint fl_hip_joint: axis 1.0 0.0 -0.0 -> 1.0 0.0 0.0; limit lower=-1.570796 upper=1.570796 effort=2.94 velocity=5.0 -> lower=-2.356194 upper=0.785398 effort=2.94 velocity=5.0
- joint fl_knee_joint: axis 1.0 0.0 -0.0 -> 1.0 0.0 0.0; limit lower=-2.356194 upper=0.523599 effort=2.94 velocity=5.0 -> lower=-1.570796 upper=1.570796 effort=2.94 velocity=5.0
- joint fl_shoulder_joint: limit lower=0.785398 upper=3.926991 effort=2.94 velocity=5.0 -> lower=-1.832596 upper=0.785398 effort=2.94 velocity=5.0; origin xyz=-0.055401 0.046222 -0.009000 rpy=0 0 -1.570796 -> xyz=-0.041500 0.049000 0.026000 rpy=0 0 0.0
- joint fr_hip_joint: axis 1.0 0.0 -0.0 -> 1.0 0.0 0.0; limit lower=-1.570796 upper=1.570796 effort=2.94 velocity=5.0 -> lower=-2.356194 upper=0.785398 effort=2.94 velocity=5.0
- joint fr_knee_joint: axis 1.0 0.0 -0.0 -> 1.0 0.0 0.0; limit lower=-2.356194 upper=0.523599 effort=2.94 velocity=5.0 -> lower=-1.570796 upper=1.570796 effort=2.94 velocity=5.0
- joint fr_shoulder_joint: limit lower=-0.785398 upper=2.356194 effort=2.94 velocity=5.0 -> lower=-0.785398 upper=1.832596 effort=2.94 velocity=5.0; origin xyz=0.055401 0.046222 -0.009000 rpy=0 0 -1.570796 -> xyz=0.041500 0.049000 0.026000 rpy=0 0 0.0

Commit message: feat(sim): leg-assembly normalization + standalone servos align URDF
Fixes two compounding bugs that put the legs in the wrong place in
PyBullet: (1) shoulder joint origin was at the mounting tab instead
of the rotation axis (38mm off), and (2) FaceHuggerLegAssembly's
90°-about-Z world rotation wasn't compensated for, leaving meshes
and joint axes 90° off.

Exporter (Phase E)
- Compute R_la = leg-assembly's 3x3 world rotation; pass into
  collect_joints() and apply to axis_dir / axis_origin for joints
  owned by FaceHuggerLegAssembly. JSON now carries world-aligned
  joint data.
- Convert all leg-assembly-internal body-rule entries to combined-rule
  (single-part). Combined-rule already bakes vertices in world frame,
  so this implicitly normalizes mesh orientation. Add `landmark_occurrence`
  field to scope landmark lookups (needed when the same name exists in
  multiple occurrences, e.g. LegMountFixedPoint in both brackets).
- Drop servo bake-ins from leg_shoulder_L.stl and leg_lower.stl;
  servo.stl is now standalone and instanced 12x by the URDF generator.
- Add `leg_assembly_normalization` block to JSON + paragraph to TXT.

URDF generator (Phases G + H + I)
- Per-corner shoulder placement: origin = LegMountPointXX_world +
  Rz(rpy_z_deg) * side_offset, where side_offset is computed from
  the JSON's BodyToLink1Point and per-bracket LegMountFixedPoint
  world positions. Rotation axis now correctly at BodyToLink1Point.
- R-pair joint axis flip: hip/knee axis (0,1,0) -> (0,-1,0) with
  negate-and-swap limits, so hip=-40 knee=-60 drops every leg
  uniformly (no per-side hacks for downstream consumers).
- Link2/Link3 mesh visual rpy = (0,π,0) for R pair (shared meshes
  need rotation since they're not separately mirrored). CoM rotates
  with the mesh.
- 12 standalone servo visuals (4 shoulder + 4 hip + 4 knee). Per-role
  rpy computed dynamically from JSON: M_role = R_role · R_servo1^T,
  yielding rpy=(-π/2, 0, 0) for hip and (0, -π/2, -π/2) for knee, so
  the shoulder-baked mesh's +Z shaft rotates to world +Y. R-pair
  position X-flipped only (no rotation — servo is the same physical
  part on every leg).

Tooling
- view_urdf.py: minimal PyBullet viewer (load + stance + step). No IK,
  no gait, no settle. Mouse-orbit only.
- URDF_PIPELINE.md: end-to-end documentation of how the pipeline
  works (re-origining, construction-point dual roles, R_la math,
  per-role servo rpy, diagonal-pair scheme).
- ALIGNMENT_FIX_PLAN.md: living plan that drove this change. Phase J
  (simulate_v2 FK rewrite) noted as next step.

Verified via PyBullet FK at zero joint angles: all 4 legs symmetric
at world (±57.9, ±46.2, -9.0) for the shoulder axis, post-norm
hip/knee axes = (0,1,0) for L pair / (0,-1,0) for R pair.

Co-Authored-By: Claude Opus 4.7 (1M context) <noreply@anthropic.com>

File: code/simulation/facehugger.urdf (robot description, URDF)
Before this commit: robot facehugger, 13 links, 12 joints
Links:
- link bl_link1: geometry collision mesh filename=exported_meshes/leg_shoulder_R.stl scale=0.001 0.001 0.001; visual mesh filename=exported_meshes/leg_shoulder_R.stl scale=0.001 0.001 0.001
- link bl_link3: geometry collision mesh filename=exported_meshes/leg_lower.stl scale=0.001 0.001 0.001; visual mesh filename=exported_meshes/leg_lower.stl scale=0.001 0.001 0.001
- link br_link1: geometry collision mesh filename=exported_meshes/leg_shoulder_L.stl scale=0.001 0.001 0.001; visual mesh filename=exported_meshes/leg_shoulder_L.stl scale=0.001 0.001 0.001
- link br_link3: geometry collision mesh filename=exported_meshes/leg_lower.stl scale=0.001 0.001 0.001; visual mesh filename=exported_meshes/leg_lower.stl scale=0.001 0.001 0.001
- link fl_link1: geometry collision mesh filename=exported_meshes/leg_shoulder_L.stl scale=0.001 0.001 0.001; visual mesh filename=exported_meshes/leg_shoulder_L.stl scale=0.001 0.001 0.001
- link fl_link3: geometry collision mesh filename=exported_meshes/leg_lower.stl scale=0.001 0.001 0.001; visual mesh filename=exported_meshes/leg_lower.stl scale=0.001 0.001 0.001
- link fr_link1: geometry collision mesh filename=exported_meshes/leg_shoulder_R.stl scale=0.001 0.001 0.001; visual mesh filename=exported_meshes/leg_shoulder_R.stl scale=0.001 0.001 0.001
- link fr_link3: geometry collision mesh filename=exported_meshes/leg_lower.stl scale=0.001 0.001 0.001; visual mesh filename=exported_meshes/leg_lower.stl scale=0.001 0.001 0.001
Joints:
- joint bl_hip_joint: axis 1.0 0.0 0.0 -> -1.1796119636642283e-16 -1.000000000000004 -2.428612866511427e-17; limit lower=-2.356194 upper=0.785398 effort=2.94 velocity=5.0 -> lower=-0.785398 upper=2.356194 effort=2.94 velocity=5.0; origin xyz=0.022595 0.050920 0.014446 rpy=0 0 0.0 -> xyz=0.050920 0.022595 0.014446 rpy=0 0 0.0
- joint bl_knee_joint: axis 1.0 0.0 0.0 -> -1.1796119636642283e-16 -1.000000000000004 -2.428612866511427e-17; origin xyz=0.000005 0.094700 0.000000 rpy=0 0 0.0 -> xyz=0.094700 0.000005 0.000000 rpy=0 0 0.0
- joint bl_shoulder_joint: axis 0.0 0.0 1.0 -> 2.774184853852289e-17 -2.9924197261652035e-17 1.0000000000000002; origin xyz=-0.041500 -0.049000 0.026000 rpy=0 0 3.141593 -> xyz=-0.057901 -0.046222 -0.009000 rpy=0 0 3.141593
- joint br_hip_joint: axis 1.0 0.0 0.0 -> 1.1796119636642283e-16 1.000000000000004 2.428612866511427e-17; origin xyz=0.022595 0.050920 0.014446 rpy=0 0 0.0 -> xyz=-0.050920 0.022595 0.014446 rpy=0 0 0.0
- joint br_knee_joint: axis 1.0 0.0 0.0 -> 1.1796119636642283e-16 1.000000000000004 2.428612866511427e-17; origin xyz=0.000005 0.094700 0.000000 rpy=0 0 0.0 -> xyz=-0.094700 0.000005 0.000000 rpy=0 0 0.0
- joint br_shoulder_joint: axis 0.0 0.0 1.0 -> 2.774184853852289e-17 -2.9924197261652035e-17 1.0000000000000002; origin xyz=0.041500 -0.049000 0.026000 rpy=0 0 3.141593 -> xyz=0.057901 -0.046222 -0.009000 rpy=0 0 3.141593
- joint fl_hip_joint: axis 1.0 0.0 0.0 -> 1.1796119636642283e-16 1.000000000000004 2.428612866511427e-17; origin xyz=0.022595 0.050920 0.014446 rpy=0 0 0.0 -> xyz=-0.050920 0.022595 0.014446 rpy=0 0 0.0
- joint fl_knee_joint: axis 1.0 0.0 0.0 -> 1.1796119636642283e-16 1.000000000000004 2.428612866511427e-17; origin xyz=0.000005 0.094700 0.000000 rpy=0 0 0.0 -> xyz=-0.094700 0.000005 0.000000 rpy=0 0 0.0
- joint fl_shoulder_joint: axis 0.0 0.0 1.0 -> 2.774184853852289e-17 -2.9924197261652035e-17 1.0000000000000002; origin xyz=-0.041500 0.049000 0.026000 rpy=0 0 0.0 -> xyz=-0.057901 0.046222 -0.009000 rpy=0 0 0.0
- joint fr_hip_joint: axis 1.0 0.0 0.0 -> -1.1796119636642283e-16 -1.000000000000004 -2.428612866511427e-17; limit lower=-2.356194 upper=0.785398 effort=2.94 velocity=5.0 -> lower=-0.785398 upper=2.356194 effort=2.94 velocity=5.0; origin xyz=0.022595 0.050920 0.014446 rpy=0 0 0.0 -> xyz=0.050920 0.022595 0.014446 rpy=0 0 0.0
- joint fr_knee_joint: axis 1.0 0.0 0.0 -> -1.1796119636642283e-16 -1.000000000000004 -2.428612866511427e-17; origin xyz=0.000005 0.094700 0.000000 rpy=0 0 0.0 -> xyz=0.094700 0.000005 0.000000 rpy=0 0 0.0
- joint fr_shoulder_joint: axis 0.0 0.0 1.0 -> 2.774184853852289e-17 -2.9924197261652035e-17 1.0000000000000002; origin xyz=0.041500 0.049000 0.026000 rpy=0 0 0.0 -> xyz=0.057901 0.046222 -0.009000 rpy=0 0 0.0
