Commit message: chore(sim): regenerate URDF + STLs + fusion_export with rest-value fix
Re-run of the Fusion exporter (post-fix from b70b771) followed by
\`python facehugger.py urdf\`. The diff is mostly binary (STLs +
JSON), but the semantic change worth eyeballing is in
fusion_export.json:

  Link1Revolute.limits_rad.rest:    0.0  ->  -0.7853981633974483 rad
                                                (= -45 deg)
  Link2Revolute.limits_rad.rest:    0.0  ->  0.0 (no change; rest = 0)
  Link3Revolute.limits_rad.rest:    0.0  ->  0.0 (no change; rest = 0)

The URDF itself does NOT yet consume these new rest values — that's
the Convention A implementation still to land in generate_urdf.py
(tracked in MERGE_AND_CONVENTION.md section 8 item 1). So the
regenerated facehugger.urdf still uses the legacy rpy_z_deg from yaml;
the regeneration is included here to (a) prove the export+gen pipeline
runs cleanly post-merge, (b) refresh STLs against current Fusion
geometry. Convention A's actual URDF impact will be a separate PR.

Co-Authored-By: Claude Opus 4.7 (1M context) <noreply@anthropic.com>

File: code/simulation/generated/facehugger.urdf (robot description, URDF)
Before this commit: robot facehugger, 13 links, 12 joints
Links:
- link bl_link1: mass 0.144017 -> 0.150899
- link bl_link2: mass 0.173381 -> 0.162564
- link br_link1: mass 0.144017 -> 0.150899
- link br_link2: mass 0.173381 -> 0.162564
- link fl_link1: mass 0.144017 -> 0.150899
- link fl_link2: mass 0.173381 -> 0.162564
- link fr_link1: mass 0.144017 -> 0.150899
- link fr_link2: mass 0.173381 -> 0.162564
Joints:
- joint bl_hip_joint: limit lower=-0.785398 upper=2.356194 effort=2.94 velocity=5.0 -> lower=-1.570796 upper=1.570796 effort=2.94 velocity=5.0; origin xyz=0.050920 0.022595 0.014446 rpy=0 0 0.0 -> xyz=0.055920 0.022595 0.014446 rpy=0 0 0.0
- joint bl_knee_joint: origin xyz=0.094700 0.000005 0.000000 rpy=0 0 0.0 -> xyz=0.089700 0.000005 0.000000 rpy=0 0 0.0
- joint br_hip_joint: limit lower=-2.356194 upper=0.785398 effort=2.94 velocity=5.0 -> lower=-1.570796 upper=1.570796 effort=2.94 velocity=5.0; origin xyz=-0.050920 0.022595 0.014446 rpy=0 0 0.0 -> xyz=-0.055920 0.022595 0.014446 rpy=0 0 0.0
- joint br_knee_joint: origin xyz=-0.094700 0.000005 0.000000 rpy=0 0 0.0 -> xyz=-0.089700 0.000005 0.000000 rpy=0 0 0.0
- joint fl_hip_joint: limit lower=-2.356194 upper=0.785398 effort=2.94 velocity=5.0 -> lower=-1.570796 upper=1.570796 effort=2.94 velocity=5.0; origin xyz=-0.050920 0.022595 0.014446 rpy=0 0 0.0 -> xyz=-0.055920 0.022595 0.014446 rpy=0 0 0.0
- joint fl_knee_joint: origin xyz=-0.094700 0.000005 0.000000 rpy=0 0 0.0 -> xyz=-0.089700 0.000005 0.000000 rpy=0 0 0.0
- joint fr_hip_joint: limit lower=-0.785398 upper=2.356194 effort=2.94 velocity=5.0 -> lower=-1.570796 upper=1.570796 effort=2.94 velocity=5.0; origin xyz=0.050920 0.022595 0.014446 rpy=0 0 0.0 -> xyz=0.055920 0.022595 0.014446 rpy=0 0 0.0
- joint fr_knee_joint: origin xyz=0.094700 0.000005 0.000000 rpy=0 0 0.0 -> xyz=0.089700 0.000005 0.000000 rpy=0 0 0.0

Commit message: refactor(urdf): clean link/joint names
Joint names now follow the Fusion-aligned `{leg_id}_link{1,2,3}_joint`
pattern (was `{leg_id}_{shoulder,hip,knee}_joint`). Link names are
unchanged at `{leg_id}_link{1,2,3}` — they already matched the CAD's
`Link1L:1` / `Link2L:1` / `Link3L:1` component names.

  Link names:  base_link
               {leg_id}_link1, {leg_id}_link2, {leg_id}_link3   (12 leg links)
  Joint names: {leg_id}_link1_joint, {leg_id}_link2_joint, {leg_id}_link3_joint

The semantic mapping link1=shoulder, link2=hip, link3=knee now lives
solely in helpers._joint_type_from_name (substring-match on `link1` /
`link2` / `link3`). Callers that speak in stance keys
(`stance["shoulder"]` etc.) are unaffected.

Behaviour change: none. PyBullet, Blender visualizers, IK math, and
gait targets all produce the same physical motion as before — they
just look up joints by the new names.

Files updated:
  - generate_urdf.py: _JOINT_TOPOLOGY urdf_name "shoulder/hip/knee" ->
                      "link1/link2/link3"
  - kinematics.py: build_config joint lookups by new names
  - gaits.py: gait_joint_targets dict keys
  - helpers.py: _joint_type_from_name substring match
  - teleop.py, terrain.py: same dict-key change so the
                          "Not yet integrated" files don't drift

Regenerated facehugger.urdf included to verify the new joint names
land in the XML and the link/joint chain still resolves cleanly.

Co-Authored-By: Claude Opus 4.7 (1M context) <noreply@anthropic.com>

File: code/simulation/generated/facehugger.urdf (robot description, URDF)
Before this commit: robot facehugger, 13 links, 12 joints
Joints:
- removed joint bl_hip_joint
- removed joint bl_knee_joint
- removed joint bl_shoulder_joint
- removed joint br_hip_joint
- removed joint br_knee_joint
- removed joint br_shoulder_joint
- removed joint fl_hip_joint
- removed joint fl_knee_joint
- removed joint fl_shoulder_joint
- removed joint fr_hip_joint
- removed joint fr_knee_joint
- removed joint fr_shoulder_joint
- added joint bl_link1_joint: type revolute, parent base_link, child bl_link1, origin xyz=-0.057901 -0.046222 -0.009000 rpy=0 0 3.141593, axis 2.774184853852289e-17 -2.9924197261652035e-17 1.0000000000000002, limit lower=-1.832596 upper=0.785398 effort=2.94 velocity=5.0
- added joint bl_link2_joint: type revolute, parent bl_link1, child bl_link2, origin xyz=0.055920 0.022595 0.014446 rpy=0 0 0.0, axis -1.1796119636642283e-16 -1.000000000000004 -2.428612866511427e-17, limit lower=-1.570796 upper=1.570796 effort=2.94 velocity=5.0
- added joint bl_link3_joint: type revolute, parent bl_link2, child bl_link3, origin xyz=0.089700 0.000005 0.000000 rpy=0 0 0.0, axis -1.1796119636642283e-16 -1.000000000000004 -2.428612866511427e-17, limit lower=-1.570796 upper=1.570796 effort=2.94 velocity=5.0
- added joint br_link1_joint: type revolute, parent base_link, child br_link1, origin xyz=0.057901 -0.046222 -0.009000 rpy=0 0 3.141593, axis 2.774184853852289e-17 -2.9924197261652035e-17 1.0000000000000002, limit lower=-0.785398 upper=1.832596 effort=2.94 velocity=5.0
- added joint br_link2_joint: type revolute, parent br_link1, child br_link2, origin xyz=-0.055920 0.022595 0.014446 rpy=0 0 0.0, axis 1.1796119636642283e-16 1.000000000000004 2.428612866511427e-17, limit lower=-1.570796 upper=1.570796 effort=2.94 velocity=5.0
- added joint br_link3_joint: type revolute, parent br_link2, child br_link3, origin xyz=-0.089700 0.000005 0.000000 rpy=0 0 0.0, axis 1.1796119636642283e-16 1.000000000000004 2.428612866511427e-17, limit lower=-1.570796 upper=1.570796 effort=2.94 velocity=5.0
- added joint fl_link1_joint: type revolute, parent base_link, child fl_link1, origin xyz=-0.057901 0.046222 -0.009000 rpy=0 0 0.0, axis 2.774184853852289e-17 -2.9924197261652035e-17 1.0000000000000002, limit lower=-1.832596 upper=0.785398 effort=2.94 velocity=5.0
- added joint fl_link2_joint: type revolute, parent fl_link1, child fl_link2, origin xyz=-0.055920 0.022595 0.014446 rpy=0 0 0.0, axis 1.1796119636642283e-16 1.000000000000004 2.428612866511427e-17, limit lower=-1.570796 upper=1.570796 effort=2.94 velocity=5.0
- added joint fl_link3_joint: type revolute, parent fl_link2, child fl_link3, origin xyz=-0.089700 0.000005 0.000000 rpy=0 0 0.0, axis 1.1796119636642283e-16 1.000000000000004 2.428612866511427e-17, limit lower=-1.570796 upper=1.570796 effort=2.94 velocity=5.0
- added joint fr_link1_joint: type revolute, parent base_link, child fr_link1, origin xyz=0.057901 0.046222 -0.009000 rpy=0 0 0.0, axis 2.774184853852289e-17 -2.9924197261652035e-17 1.0000000000000002, limit lower=-0.785398 upper=1.832596 effort=2.94 velocity=5.0
- added joint fr_link2_joint: type revolute, parent fr_link1, child fr_link2, origin xyz=0.055920 0.022595 0.014446 rpy=0 0 0.0, axis -1.1796119636642283e-16 -1.000000000000004 -2.428612866511427e-17, limit lower=-1.570796 upper=1.570796 effort=2.94 velocity=5.0
- added joint fr_link3_joint: type revolute, parent fr_link2, child fr_link3, origin xyz=0.089700 0.000005 0.000000 rpy=0 0 0.0, axis -1.1796119636642283e-16 -1.000000000000004 -2.428612866511427e-17, limit lower=-1.570796 upper=1.570796 effort=2.94 velocity=5.0

Commit message: feat(urdf): implement Convention A — shoulder rest from FL Fusion export
Bake the Fusion-defined per-joint rest into the URDF so URDF θ=0 equals
each leg's mechanical zero. Limits become symmetric ±90° about θ=0.

  FL = json["Link1Revolute"]["limits_rad"]["rest"]   (-π/4 from current CAD)
  FR = -FL
  BL = wrap_pi(FL + π)
  BR = -wrap_pi(FL + π)

URDF effects per shoulder joint:
  <axis xyz="0 0 1"/>                          uniform (Convention A)
  <origin xyz="..." rpy="0 0 {rest_rad}"/>     per-leg, derived above
  <limit lower="{min - rest}" upper="{max - rest}" .../>
                                              symmetric about 0 by design

Hip and knee joints: unchanged. Their Fusion rest is 0 in CAD, so the
URDF rpy stays 0 and the existing R-pair ±Y axis flip + X-mirror logic
is untouched.

The geometric back-of-pair flip (chassis bracket placement, shoulder
pivot positioning) used to live in yaml as `rpy_z_deg = 0|180`. It's
now derived from leg_id ("b*" = back-of-pair = 180°) via
_back_of_pair_rpy_z_deg(). Distinct from the Convention-A kinematic
shoulder rest, which is a different angle and applies to the URDF
<origin rpy>.

Yaml drops three fields (now derived from the JSON):
  - legs[].rpy_z_deg            -> from leg_id (geometric) + JSON formula (kinematic)
  - legs[].shoulder_limits_deg  -> from JSON limits shifted by FL rest
  - legs[].shoulder_neutral_deg -> identical to URDF θ=0 under Convention A

Generated URDF for current CAD (FL rest = -45°):

  fl_link1_joint:  rest=-45°,   rpy="0 0 -0.785",  limits=[-π/2, +π/2]
  fr_link1_joint:  rest=+45°,   rpy="0 0 +0.785",  limits=[-π/2, +π/2]
  bl_link1_joint:  rest=+135°,  rpy="0 0 +2.356",  limits=[-π/2, +π/2]
  br_link1_joint:  rest=-135°,  rpy="0 0 -2.356",  limits=[-π/2, +π/2]

Note: this matches the formula in MERGE_AND_CONVENTION.md §0/§4 but
NOT the rest-angle table at the top of §0 (which has FL=+135°, FR=+45°,
BR=-45°, BL=-135°). The two specs disagreed; this commit implements
the formula. Reconcile by either updating the table to match
(FL=-45°, FR=+45°, BL=+135°, BR=-135°) or negating the FL rest in
Fusion so FL=+135° comes out of JSON.

Co-Authored-By: Claude Opus 4.7 (1M context) <noreply@anthropic.com>

File: code/simulation/generated/facehugger.urdf (robot description, URDF)
Before this commit: robot facehugger, 13 links, 12 joints
Joints:
- joint bl_link1_joint: limit lower=-1.832596 upper=0.785398 effort=2.94 velocity=5.0 -> lower=-1.570796 upper=1.570796 effort=2.94 velocity=5.0; origin xyz=-0.057901 -0.046222 -0.009000 rpy=0 0 3.141593 -> xyz=-0.057901 -0.046222 -0.009000 rpy=0 0 2.356194
- joint br_link1_joint: limit lower=-0.785398 upper=1.832596 effort=2.94 velocity=5.0 -> lower=-1.570796 upper=1.570796 effort=2.94 velocity=5.0; origin xyz=0.057901 -0.046222 -0.009000 rpy=0 0 3.141593 -> xyz=0.057901 -0.046222 -0.009000 rpy=0 0 -2.356194
- joint fl_link1_joint: limit lower=-1.832596 upper=0.785398 effort=2.94 velocity=5.0 -> lower=-1.570796 upper=1.570796 effort=2.94 velocity=5.0; origin xyz=-0.057901 0.046222 -0.009000 rpy=0 0 0.0 -> xyz=-0.057901 0.046222 -0.009000 rpy=0 0 -0.785398
- joint fr_link1_joint: limit lower=-0.785398 upper=1.832596 effort=2.94 velocity=5.0 -> lower=-1.570796 upper=1.570796 effort=2.94 velocity=5.0; origin xyz=0.057901 0.046222 -0.009000 rpy=0 0 0.0 -> xyz=0.057901 0.046222 -0.009000 rpy=0 0 0.785398

Commit message: fix(urdf): swap BL/BR signs in Convention A shoulder rest formula
The previous _shoulder_rest_for() had BL and BR swapped (signs flipped
relative to what makes back legs splay outward). With FL = -π/4 from
the current CAD, the wrong formula gave BL=+135° / BR=-135°, which
sent the back legs pointing into the FRONT quadrants — visible in
Blender as BL aiming toward the FL corner and BR toward FR.

Correct mapping (verified against Blender visualizer):

    FL =  fl_rest_rad         (= -45° from current CAD)
    FR = -fl_rest_rad         (= +45°)
    BL = -wrap_pi(FL + π)     (= -135°)   ← sign flipped from previous
    BR =  wrap_pi(FL + π)     (= +135°)   ← sign flipped from previous

All four legs now splay outward into their respective body quadrants:
  FL at (-X, +Y) corner pointing toward -45° in world,
  FR at (+X, +Y) toward +45°,
  BL at (-X, -Y) toward -135°,
  BR at (+X, -Y) toward +135°.

URDF deltas (all 4 shoulder joints):
  fl_link1_joint  rpy="0 0 -0.785"   (unchanged: -45°)
  fr_link1_joint  rpy="0 0 +0.785"   (unchanged: +45°)
  bl_link1_joint  rpy="0 0 -2.356"   (was +2.356, now -2.356)
  br_link1_joint  rpy="0 0 +2.356"   (was -2.356, now +2.356)

MERGE_AND_CONVENTION.md §0 quick-ref + §4 derivation table updated to
match. Added a one-paragraph note about the previous bug for future
context.

Co-Authored-By: Claude Opus 4.7 (1M context) <noreply@anthropic.com>

File: code/simulation/generated/facehugger.urdf (robot description, URDF)
Before this commit: robot facehugger, 13 links, 12 joints
Joints:
- joint bl_link1_joint: origin xyz=-0.057901 -0.046222 -0.009000 rpy=0 0 2.356194 -> xyz=-0.057901 -0.046222 -0.009000 rpy=0 0 -2.356194
- joint br_link1_joint: origin xyz=0.057901 -0.046222 -0.009000 rpy=0 0 -2.356194 -> xyz=0.057901 -0.046222 -0.009000 rpy=0 0 2.356194

Commit message: feat(animation): aim link1 bone-Y at foot tip + body_ctrl + Link3TipPoint
Aim link1's bone-Y at the foot tip in the horizontal plane, instead of
at the hip pivot. Without this, shoulder→hip and shoulder→foot differ
by ~19° at URDF rest, and Damped Track yaws link1 by that angle when
the dep graph evaluates — visually contorting the rest pose by ~88 mm
at the foot. With foot-tip aim, Damped Track is identity at rest
(yaw-only mismatch 0.014° on all 4 legs) and foot_target sits on the
visible foot mesh tip (delta 0.212 mm).

Joint axis for link1 stays world +Z; the existing perpendicular-to-
joint-axis projection in `_bone_endpoints_world_mm` keeps bone-local Z
= world +Z. Alignment invariant preserved (max bone-Z error 0.0242°,
float-precision noise on FL link2/link3; fl_link1 itself went from
~0.014° to 0.0000°).

Auto-yaw still fires on foot_target movement: dynamic verify shows
fl_link1 yaws -14.478° when foot_target_fl moves +50 mm in world X.
Damped Track's effective rotation through LIMIT_ROTATION's X/Y locks
is identity at rest and nonzero on movement — exactly the intended
behaviour.

Other changes bundled in:

- body_ctrl Empty (CUBE, 80 mm) in new Controls collection. Armature
  reparented to body_ctrl and hidden by default; animator drags the
  cube to translate the rig, foot Empties (unparented, world space)
  stay planted, IK + Damped Track keep legs reaching back.
- Loader switched from Link3TipAxis (construction axis) to Link3TipPoint
  (construction point) per the CAD refactor. Reads `pos_mm` from
  `points[]` instead of `origin_mm` from `axes[]`.
- Foot tip source: prefer FOOT_TIP_FALLBACK_IN_LINK3_FRAME_M (URDF
  metadata, mesh max-+Y centroid) over JSON Link3TipPoint. Warn at
  rig-build if they disagree by > 5 mm — current CAD point is 57.69 mm
  off, so the warning fires until the construction point gets moved
  to coincide with the leg_lower.stl tip.
- IK Z limits on link2/link3 (`use_ik_limit_z` + `ik_min_z`/`ik_max_z`
  from URDF) so the IK solver respects URDF range during the iterative
  solve, not just LIMIT_ROTATION's post-hoc clamp.
- LIMIT_ROTATION extended: X and Y locked to 0 on every joint bone,
  forcing 1-DOF around bone-local Z.
- foot_ik now copies foot_target exactly (use_offset=False); the
  static-offset trick was removed.
- Per-leg foot tip mirror via `_foot_tip_for_leg`: R-side legs (FR, BL)
  get the X component of the link3-frame foot tip negated to match
  their mirrored leg_lower.stl visual (rpy=(0, π, 0)).

CAD side (cad/scripts/...ExportBodiesToURDF.py): Link3TipAxis removed
from CONSTRUCTION_AXES whitelist, Link3TipPoint added to
CONSTRUCTION_POINTS. Re-export updates fusion_export.json/.txt and
regenerates QuadrupedBody.stl + facehugger.urdf accordingly.

New rig-build diagnostics (printed at every run):
  * `Damped Track rest-identity check` — 3D + yaw-only angle for each
    link1, confirming Damped Track is identity at rest.
  * `foot_target vs mesh tip` — per-leg distance from the foot_target
    Empty to leg_lower mesh max-+Y centroid (0 = on the mesh).
  * `bone-Z alignment per bone` — angle between bone-local Z and URDF
    joint axis for every joint bone.
  * `auto-yaw` — programmatic dynamic check (move foot_target, read
    resolved bone-Y rotation).

Co-Authored-By: Claude Opus 4.7 (1M context) <noreply@anthropic.com>

File: code/simulation/generated/facehugger.urdf (robot description, URDF)
Before this commit: robot facehugger, 13 links, 12 joints
Links:
- link base_link: mass 0.631194 -> 0.629946

Commit message: fix(urdf): snap near-zero axis components to 0 + renormalize
Fusion-derived joint axes carry FP dust on the should-be-zero columns
(e.g. [2.77e-17, -2.99e-17, 1.0000000000000002]), which some URDF
consumers reject as non-unit or treat as truly off-axis. Add a
clean_axis helper and call it in URDF.joint so emitted <axis xyz=...>
elements are exact unit vectors like "0.0 0.0 1.0".

Co-Authored-By: Claude Opus 4.7 (1M context) <noreply@anthropic.com>

File: code/simulation/generated/facehugger.urdf (robot description, URDF)
Before this commit: robot facehugger, 13 links, 12 joints
Joints:
- joint bl_link1_joint: axis 2.774184853852289e-17 -2.9924197261652035e-17 1.0000000000000002 -> 0.0 0.0 1.0
- joint bl_link2_joint: axis -1.1796119636642283e-16 -1.000000000000004 -2.428612866511427e-17 -> 0.0 -1.0 0.0
- joint bl_link3_joint: axis -1.1796119636642283e-16 -1.000000000000004 -2.428612866511427e-17 -> 0.0 -1.0 0.0
- joint br_link1_joint: axis 2.774184853852289e-17 -2.9924197261652035e-17 1.0000000000000002 -> 0.0 0.0 1.0
- joint br_link2_joint: axis 1.1796119636642283e-16 1.000000000000004 2.428612866511427e-17 -> 0.0 1.0 0.0
- joint br_link3_joint: axis 1.1796119636642283e-16 1.000000000000004 2.428612866511427e-17 -> 0.0 1.0 0.0
- joint fl_link1_joint: axis 2.774184853852289e-17 -2.9924197261652035e-17 1.0000000000000002 -> 0.0 0.0 1.0
- joint fl_link2_joint: axis 1.1796119636642283e-16 1.000000000000004 2.428612866511427e-17 -> 0.0 1.0 0.0
- joint fl_link3_joint: axis 1.1796119636642283e-16 1.000000000000004 2.428612866511427e-17 -> 0.0 1.0 0.0
- joint fr_link1_joint: axis 2.774184853852289e-17 -2.9924197261652035e-17 1.0000000000000002 -> 0.0 0.0 1.0
- joint fr_link2_joint: axis -1.1796119636642283e-16 -1.000000000000004 -2.428612866511427e-17 -> 0.0 -1.0 0.0
- joint fr_link3_joint: axis -1.1796119636642283e-16 -1.000000000000004 -2.428612866511427e-17 -> 0.0 -1.0 0.0
