Commit message: feat(urdf): shoulder three-flip on R-side + new-CAD pipeline updates
CAD redesign brought a smaller chassis (body track 83→68 mm × 98→92 mm),
raised shoulder pivot (BodyToLink1Point Z −4.2 → +41.8 mm), two new
structural bodies (MiddleBridge, BehindBridge) under QuadrupedBody:1,
and asymmetric Fusion shoulder limits ([-97°, +25°] about FL rest).

Generator changes:
- Apply the same axis-negation + limit negate-and-swap pattern that
  hip/knee already use on R-side (FR + BL) to the shoulder joint.
  Without this, asymmetric Fusion limits get applied identically to
  every leg, leaving FR/BL with a mirrored sweep window. Convention A
  is preserved — the per-leg <origin rpy> still places URDF θ=0 at
  each leg's mechanical zero.
- Add MiddleBridge + BehindBridge to the chassis combined-rule in
  ExportBodiesToURDF so QuadrupedBody.stl includes the new structural
  members alongside the original frame and LipoCage.

Docs (doc/animation-pipeline/urdf-conventions.md): new section laying
out frames (body, mount-point, joint), the four-leg part-reuse table,
the "axis points along servo base-bottom → horn" convention, and why
R-side legs need axis negation + limit negate-and-swap.

Bumps .python-version from `system` (uv warning) to `3.12`.

Co-Authored-By: Claude Opus 4.7 (1M context) <noreply@anthropic.com>

File: code/simulation/generated/facehugger.urdf (robot description, URDF)
Before this commit: robot facehugger, 13 links, 12 joints
Links:
- link base_link: mass 0.629946 -> 0.565732
- link bl_link1: mass 0.150899 -> 0.134355
- link bl_link2: mass 0.162564 -> 0.152739
- link bl_link3: mass 0.111653 -> 0.136030
- link br_link1: mass 0.150899 -> 0.134355
- link br_link2: mass 0.162564 -> 0.152739
- link br_link3: mass 0.111653 -> 0.136030
- link fl_link1: mass 0.150899 -> 0.134355
- link fl_link2: mass 0.162564 -> 0.152739
- link fl_link3: mass 0.111653 -> 0.136030
- link fr_link1: mass 0.150899 -> 0.134355
- link fr_link2: mass 0.162564 -> 0.152739
- link fr_link3: mass 0.111653 -> 0.136030
Joints:
- joint bl_link1_joint: axis 0.0 0.0 1.0 -> 0.0 0.0 -1.0; limit lower=-1.570796 upper=1.570796 effort=2.94 velocity=5.0 -> lower=-1.570796 upper=0.907571 effort=2.94 velocity=5.0; origin xyz=-0.057901 -0.046222 -0.009000 rpy=0 0 -2.356194 -> xyz=-0.050401 -0.043222 0.036844 rpy=0 0 -2.356194
- joint bl_link2_joint: limit lower=-1.570796 upper=1.570796 effort=2.94 velocity=5.0 -> lower=-0.785398 upper=0.785398 effort=2.94 velocity=5.0; origin xyz=0.055920 0.022595 0.014446 rpy=0 0 0.0 -> xyz=0.055920 0.022595 -0.031598 rpy=0 0 0.0
- joint bl_link3_joint: origin xyz=0.089700 0.000005 0.000000 rpy=0 0 0.0 -> xyz=0.060700 0.000005 0.000000 rpy=0 0 0.0
- joint br_link1_joint: limit lower=-1.570796 upper=1.570796 effort=2.94 velocity=5.0 -> lower=-0.907571 upper=1.570796 effort=2.94 velocity=5.0; origin xyz=0.057901 -0.046222 -0.009000 rpy=0 0 2.356194 -> xyz=0.050401 -0.043222 0.036844 rpy=0 0 2.356194
- joint br_link2_joint: limit lower=-1.570796 upper=1.570796 effort=2.94 velocity=5.0 -> lower=-0.785398 upper=0.785398 effort=2.94 velocity=5.0; origin xyz=-0.055920 0.022595 0.014446 rpy=0 0 0.0 -> xyz=-0.055920 0.022595 -0.031598 rpy=0 0 0.0
- joint br_link3_joint: origin xyz=-0.089700 0.000005 0.000000 rpy=0 0 0.0 -> xyz=-0.060700 0.000005 0.000000 rpy=0 0 0.0
- joint fl_link1_joint: limit lower=-1.570796 upper=1.570796 effort=2.94 velocity=5.0 -> lower=-0.907571 upper=1.570796 effort=2.94 velocity=5.0; origin xyz=-0.057901 0.046222 -0.009000 rpy=0 0 -0.785398 -> xyz=-0.050401 0.043222 0.036844 rpy=0 0 -0.785398
- joint fl_link2_joint: limit lower=-1.570796 upper=1.570796 effort=2.94 velocity=5.0 -> lower=-0.785398 upper=0.785398 effort=2.94 velocity=5.0; origin xyz=-0.055920 0.022595 0.014446 rpy=0 0 0.0 -> xyz=-0.055920 0.022595 -0.031598 rpy=0 0 0.0
- joint fl_link3_joint: origin xyz=-0.089700 0.000005 0.000000 rpy=0 0 0.0 -> xyz=-0.060700 0.000005 0.000000 rpy=0 0 0.0
- joint fr_link1_joint: axis 0.0 0.0 1.0 -> 0.0 0.0 -1.0; limit lower=-1.570796 upper=1.570796 effort=2.94 velocity=5.0 -> lower=-1.570796 upper=0.907571 effort=2.94 velocity=5.0; origin xyz=0.057901 0.046222 -0.009000 rpy=0 0 0.785398 -> xyz=0.050401 0.043222 0.036844 rpy=0 0 0.785398
- joint fr_link2_joint: limit lower=-1.570796 upper=1.570796 effort=2.94 velocity=5.0 -> lower=-0.785398 upper=0.785398 effort=2.94 velocity=5.0; origin xyz=0.055920 0.022595 0.014446 rpy=0 0 0.0 -> xyz=0.055920 0.022595 -0.031598 rpy=0 0 0.0
- joint fr_link3_joint: origin xyz=0.089700 0.000005 0.000000 rpy=0 0 0.0 -> xyz=0.060700 0.000005 0.000000 rpy=0 0 0.0

Commit message: chore(cad): regenerate URDF + Fusion export — longer link2, wider hip range
Picks up the latest Fusion export and a URDF regen:

- **link2 geometry**: source Link2.stl + re-origined
  exported_meshes/leg_upper.stl updated. URDF Link2ToLink3Point shifts
  from -106.620 to -121.620 mm in the leg-assembly-local frame (link2
  ~15 mm longer); link3 joint origin moves accordingly
  (-0.059700 → -0.074700 m). Link3.stl + leg_lower.stl also refreshed.
- **Wider hip range of motion**: link2 joint <limit> on all 4 legs
  goes ±45° → ±60° (-1.047198 .. 1.047198 rad). link1 stays
  [-52°, +90°], link3 stays ±90°.
- **link2 inertials updated** for the new geometry: mass per leg
  link2 0.134863 → 0.151342 kg, with refreshed COM and inertia
  tensors. (Body / link1 / link3 inertials unchanged.)
- fusion_export.json/txt are byte-consistent with the prior Fusion
  add-in run that added BodyBottomPoint to the construction-point
  whitelist and renamed the source assembly to FaceHuggerLegAssembly:1
  (rig builder already consumes BodyBottomPoint via
  urdf_to_blender_rigged.py's load_body_bottom_point).

Downstream impact:
- Blender rig (LIMIT_ROTATION constraints) inherits the new ±60° hip
  range on the next `python code/simulation/facehugger.py blender
  --rigged` rebuild; existing in-flight poses in fh_rigged_latest.blend
  are unaffected.
- Existing poses.json / clips author angles within previously valid
  ranges, so they remain valid (a hip authored at -45° still sits
  inside the new ±60° envelope).

Co-Authored-By: Claude Opus 4.7 (1M context) <noreply@anthropic.com>

File: code/simulation/generated/facehugger.urdf (robot description, URDF)
Before this commit: robot facehugger, 13 links, 12 joints
Links:
- link bl_link2: mass 0.141725 -> 0.151342
- link bl_link3: mass 0.131103 -> 0.127150
- link br_link2: mass 0.141725 -> 0.151342
- link br_link3: mass 0.131103 -> 0.127150
- link fl_link2: mass 0.141725 -> 0.151342
- link fl_link3: mass 0.131103 -> 0.127150
- link fr_link2: mass 0.141725 -> 0.151342
- link fr_link3: mass 0.131103 -> 0.127150
Joints:
- joint bl_link2_joint: limit lower=-0.785398 upper=0.785398 effort=2.94 velocity=5.0 -> lower=-1.047198 upper=1.047198 effort=2.94 velocity=5.0
- joint bl_link3_joint: origin xyz=0.059700 0.000205 0.000000 rpy=0 0 0.0 -> xyz=0.074700 0.000205 0.000000 rpy=0 0 0.0
- joint br_link2_joint: limit lower=-0.785398 upper=0.785398 effort=2.94 velocity=5.0 -> lower=-1.047198 upper=1.047198 effort=2.94 velocity=5.0
- joint br_link3_joint: origin xyz=-0.059700 0.000205 0.000000 rpy=0 0 0.0 -> xyz=-0.074700 0.000205 0.000000 rpy=0 0 0.0
- joint fl_link2_joint: limit lower=-0.785398 upper=0.785398 effort=2.94 velocity=5.0 -> lower=-1.047198 upper=1.047198 effort=2.94 velocity=5.0
- joint fl_link3_joint: origin xyz=-0.059700 0.000205 0.000000 rpy=0 0 0.0 -> xyz=-0.074700 0.000205 0.000000 rpy=0 0 0.0
- joint fr_link2_joint: limit lower=-0.785398 upper=0.785398 effort=2.94 velocity=5.0 -> lower=-1.047198 upper=1.047198 effort=2.94 velocity=5.0
- joint fr_link3_joint: origin xyz=0.059700 0.000205 0.000000 rpy=0 0 0.0 -> xyz=0.074700 0.000205 0.000000 rpy=0 0 0.0

Commit message: chore(cad): finalize link2 geometry — refined inertials + slicer pack
Iterates on the link2 work from 3404048:

- Refined Link2.stl geometry (source STL + re-origined
  exported_meshes/leg_upper.stl regenerated).
- URDF link2 inertials updated for the new geometry: mass per leg
  link2 0.151342 → 0.149366 kg, with refreshed COM (~0.4 mm shift)
  and inertia tensors. Joint limits, link2 length, and other links'
  inertials unchanged from 3404048.
- fusion_export.json/txt: Link3TipPoint local pos refreshed (-13.035
  → -13.012 mm in link3 frame); mass + COM picked up on
  FaceHuggerLegAssembly:1; LegBaseServoEnclosure:3 now [hidden].
- Prusa slicer pack rebuilt for the new Link2 mesh
  (FHLegsLink1and2.3mf: 124878 → 126409 bytes).

cad/print_export.txt timestamp drift restored (no semantic change).

Co-Authored-By: Claude Opus 4.7 (1M context) <noreply@anthropic.com>

File: code/simulation/generated/facehugger.urdf (robot description, URDF)
Before this commit: robot facehugger, 13 links, 12 joints
Links:
- link bl_link2: mass 0.151342 -> 0.149366
- link br_link2: mass 0.151342 -> 0.149366
- link fl_link2: mass 0.151342 -> 0.149366
- link fr_link2: mass 0.151342 -> 0.149366

Commit message: fix(urdf): restore missing FR/BL shoulder servo visuals
The right-side shoulder servo position was looked up at the wrong occurrence
path (MotorMountR:1/LegBaseServoEnclosure(Mirror):1), which does not exist in
the Fusion export; the mirrored servo is MotorMountR:1/Servo_Mouser_Model(Mirror):1.
The lookup returned None, so shoulder_servo_R_offset was None and the FR/BL
chassis shoulder servos were skipped, leaving base_link with only two of four.
Correct the path and warn instead of silently skipping when a servo datum is
missing. Regenerated URDF now emits all four shoulder servos.

Co-Authored-By: Claude Opus 4.7 (1M context) <noreply@anthropic.com>

File: code/simulation/generated/facehugger.urdf (robot description, URDF)
Before this commit: robot facehugger, 13 links, 12 joints
Links:
- link base_link: geometry collision mesh filename=exported_meshes/QuadrupedBody.stl scale=0.001 0.001 0.001; visual mesh filename=exported_meshes/QuadrupedBody.stl scale=0.001 0.001 0.001

Commit message: fix(sim): account for unmodelled electronics in base_link mass
Add base_link.extra_mass_kg override in facehugger_config.yaml (0.239 kg from
the current BOM: ESP32, PCA9685, mux, IMU, 5×ToF, OLED, 1000mAh 2S LiPo, buck,
BMS, XT60×4, switch, wiring) and have generate_urdf.py fold it into the
Fusion-derived chassis mass. base_link goes 0.566 → 0.805 kg, closer to real.

COM/inertia stay Fusion's: the electronics cluster is roughly co-located with
the chassis centroid, and the static-torque change from skipping a COM shift
is within the noise of this check.

Note: this is the BOM-accuracy fix, not a fix for the standstill SIL red.
That red is a hand-calibrated-firmware-NEUTRAL vs perfect-sim-joints artifact:
BR's thigh is +10° off perfect mirror (calibrated for real gear backlash), so
in the ideal sim BR floats and the bl-fr diagonal carries everything and
saturates at the 2.94 N·m servo ceiling. Mass at 0.57 / 0.80 / 0.98 kg all
gives the same red — confirmed not a load problem.

Co-Authored-By: Claude Opus 4.7 (1M context) <noreply@anthropic.com>

File: code/simulation/generated/facehugger.urdf (robot description, URDF)
Before this commit: robot facehugger, 13 links, 12 joints
Links:
- link base_link: mass 0.565732 -> 0.804732

Commit message: fix(sim): add shoulder-servo mass to base_link, lock crab against regression
The 4 shoulder servos (~0.06 kg each, 0.240 kg total) are nailed to the chassis
in Fusion as massless visuals — invisible to the URDF mass budget. Roll them
into base_link.extra_mass_kg alongside the electronics; placement at the four
corners is symmetric, so COM stays at the chassis centroid. base_link goes
0.805 -> 1.045 kg, closer to the real platform mass. The 8 leg servos may or
may not be in their link masses already (Fusion side TBD) — separate audit.

Crab audit vs pre-branch (commit 7debf36): no regression. The FL Change B and
BR un-mirror only touched the HIP path in translateToServo; pure-X crab in
tickGait keeps the shoulder at NEUTRAL (fwdContrib=0, yawDir*0=0), so every
shoulder lands at servo 90 by construction. Lateral motion still rides on the
thigh sweep, whose signs and translateToServo conversion are unchanged.
Pinning this with a new SIL test so a future NEUTRAL or translateToServo edit
can't silently re-introduce shoulder motion in pure-sideways crab.

Co-Authored-By: Claude Opus 4.7 (1M context) <noreply@anthropic.com>

File: code/simulation/generated/facehugger.urdf (robot description, URDF)
Before this commit: robot facehugger, 13 links, 12 joints
Links:
- link base_link: mass 0.804732 -> 1.044732
