Commit message: Animation-flow integration: Full pipeline for playing Blender-created animations and simulating firmware faithfully (#102)
(firmware-faithful sim, clip pipeline, invert rework, and a unified facehugger CLI (#102))
Testing on the robot worked! The dance that I animated in Blender was successfully played on the robot!

---

* fix(firmware): clamp servo angle to 0-180 with warning in setServoAngle

setServoAngle() funnels every motion path (IK, pose, calibrate, future
clip player), but map() does not clamp — an out-of-range angle drove the
servo past MIN/MAX_PULSE. Only the JS-side clamp protected servos; manual
T:4, the app, or any future tool bypassed it.

Add constrain(angle, 0, 180) at this single chokepoint plus a Serial
warning when a value is clamped. Verified: pio run -e upesy_wroom SUCCESS.

Co-Authored-By: Claude Opus 4.7 (1M context) <noreply@anthropic.com>

* test(animation): headless regression for bake_clip active-clip bleed

Co-Authored-By: Claude Opus 4.7 (1M context) <noreply@anthropic.com>

* fix(animation): bind target clip in bake_clip before sampling

bake_clip read the live depsgraph pose using only the target clip's
frame_range, so multi-clip Export Selected baked the active clip under
every name (export-review findings §2). Autocomplete + assign_clip +
view_layer.update() before the frame loop; restore the previously-active
clip + frame after. Regression test now GREEN.

Co-Authored-By: Claude Opus 4.7 (1M context) <noreply@anthropic.com>

* feat(animation): warn on per-frame joint deltas above threshold

Co-Authored-By: Claude Opus 4.7 (1M context) <noreply@anthropic.com>

* test(animation): verify JS export wire contract (LEG_IDS, clamp, FRAME_MS)

Co-Authored-By: Claude Opus 4.7 (1M context) <noreply@anthropic.com>

* feat(animation): warn when scene fps exceeds recommended robot-export rate

Co-Authored-By: Claude Opus 4.7 (1M context) <noreply@anthropic.com>

* fix(animation): add to_js write= param; restore dry-run file write

f5d4719 made dry_run return early before writing, silently breaking the
Export-JS-dry-run operator path. dry_run is a template-content choice, not
a write toggle. Separate the concerns: new write=True param (write=False
returns the string for tests); dry_run no longer suppresses the file write.
Test now validates the real WebSocket template via write=False.

Co-Authored-By: Claude Opus 4.7 (1M context) <noreply@anthropic.com>

* perf(animation): delta-encode JS servo stream + connection-failure alert

Only emit a servo message when its value changed from the previous frame
(cuts redundant traffic; ends the hold-at-end resend flood). Add ws.onerror
alert + onclose warning so a wrong/unreachable robot IP is visible instead
of failing silently.

Co-Authored-By: Claude Opus 4.7 (1M context) <noreply@anthropic.com>

* feat(animation): add Preview Robot Motion (BEZIER<->LINEAR) toggle

Non-destructive N-panel toggle flipping the active clip's F-curve keyframe
interpolation between BEZIER (authoring) and LINEAR (what the robot plays).
Walks the Blender 5.x layered Action API (layer -> strip -> channelbag ->
fcurves). Bezier handle data is preserved, so toggling back restores curves.

Co-Authored-By: Claude Opus 4.7 (1M context) <noreply@anthropic.com>

* chore(animation): track canonical rig via git-lfs; un-ignore exported_gaits

Add .gitattributes routing *.blend through git-lfs and track the canonical
rig fh_rigged_latest.blend (1.2 MB). Un-ignore animation/exported_gaits/ so
re-exported clips (text .js/.h/.csv) are reviewable in PRs. blend-iterations/
and *.blend1 stay ignored. Teammates run `git lfs install` once locally.

Co-Authored-By: Claude Opus 4.7 (1M context) <noreply@anthropic.com>

* docs(animation): add motion-domain CONTEXT.md + Phase-0 exporter plan

CONTEXT.md captures the clip/gait/math-space/servo-space glossary and the
clip-end (return-to-stand) decision crystallised during the grill session.
The plan is the TDD breakdown executed as T1-T9.

Co-Authored-By: Claude Opus 4.7 (1M context) <noreply@anthropic.com>

* chore(animation): headless export-all driver + re-export verified clips

export_all_clips.py re-bakes every clip via the fixed bake_clip + Layer-2
converters (no operator/scene-property dependency, runs headless). Re-export
of all 5 clips now yields 5 DISTINCT payloads — previously tiny wiggle,
wiggle and lie-down-and-stand-up were byte-identical (the bake_clip bug).

Co-Authored-By: Claude Opus 4.7 (1M context) <noreply@anthropic.com>

* docs(animation): track deferred tasks T10-T13 (IP config, heatmap, validator)

T10 robot-IP scene property; T11 heatmap rework (delta + URDF-limit + real
PyBullet torque); T12 PyBullet clip validator + facehugger.py validate
subcommand; T13 read-only info-gathering on CSV angle space (do before T12).

Co-Authored-By: Claude Opus 4.7 (1M context) <noreply@anthropic.com>

* refactor(animation): rename exported_gaits/ -> exported_clips/ (glossary fix)

The directory holds Clips (one-shot), not Gaits (looping); CONTEXT.md keeps
those distinct. Rename the dir + _exported_clips_dir helper + all references.
No .gitignore change (Phase 0 already un-ignored the path).

Co-Authored-By: Claude Opus 4.7 (1M context) <noreply@anthropic.com>

* feat(animation): bundled to_clips_header (clips_all.h + manifest)

Math-space pre-scaled clip header for the on-board clip player. Reuses the
scale-from-NEUTRAL step (not translateToServo/round, unlike the JS path);
firmware applies translateToServo at runtime. Pure-Python test asserts the
frozen contract: leg reorder FR,FL,RR,RL, scale-once, t_ms, determinism.

Co-Authored-By: Claude Opus 4.7 (1M context) <noreply@anthropic.com>

* feat(animation): to_clips_header guards (empty, t_ms order, symbol collision, u16 overflow)

Co-Authored-By: Claude Opus 4.7 (1M context) <noreply@anthropic.com>

* feat(animation): export-all driver emits clips_all.h + clips_manifest.json

Co-Authored-By: Claude Opus 4.7 (1M context) <noreply@anthropic.com>

* docs(animation): document clips_all.h pre-scale + math-space rule

Add a concrete 'Clip header' section stating clips_all.h is pre-scaled
math-space (firmware applies only translateToServo), differing from the
JS path's _frame_to_servo. Also fix the stale 'hold-at-end' reference in
the angle-conversion note: clip end is now return-to-NEUTRAL over 500ms
(code-over-docs; CONTEXT.md is authoritative).

Co-Authored-By: Claude Opus 4.7 (1M context) <noreply@anthropic.com>

* refactor(firmware): extract shared translateToServo helper (pure, native-tested)

Lift the per-leg math-space->servo switch (duplicated in tickGait/tickTrot/
tickYawRotation) into motion_math.cpp::translateToServo. Native Unity test
pins the four per-leg formulas. Gait output unchanged (verbatim copy).

Co-Authored-By: Claude Opus 4.7 (1M context) <noreply@anthropic.com>

* feat(firmware): pure clip frame interpolation (lerp/bracket/hold) + tests

Co-Authored-By: Claude Opus 4.7 (1M context) <noreply@anthropic.com>

* feat(firmware): pure clip lifecycle phase machine (PLAYING/RETURNING/DONE) + tests

Extract the clip lifecycle (return-to-NEUTRAL transition, 500ms timing,
single-frame/duration=0 edge) into a pure clipPlayerStep so every
transition is unit-tested on the host. tickClip (B4) becomes a thin
dispatcher over the returned action.

Co-Authored-By: Claude Opus 4.7 (1M context) <noreply@anthropic.com>

* fix(firmware): decouple clip test fixture from production clips_all.h

motion_math.h includes clips_all.h to get FhClipFrame, so the production
header lands in the test translation unit. The fixture previously shared
the production guard (FH_CLIPS_ALL_H) AND symbols, so it was guard-shadowed
and only compiled because the placeholder happened to copy the fixture's
clips — after INT1 (real bundle) test_clip_interp would have broken.

Fixture now uses guard FH_CLIPS_TEST_FIXTURE_H and defines ONLY its frame
arrays (types from motion_math.h), never the registry. Production keeps
guard FH_CLIPS_ALL_H but uses a distinct fh_clip_placeholder clip so its
symbols never collide with the fixture's. All 26 native tests pass; INT1
swap is now safe.

Co-Authored-By: Claude Opus 4.7 (1M context) <noreply@anthropic.com>

* feat(firmware): non-blocking setServoAngleTimed easing (Servo + Leg)

Per-Servo ease state advanced by tickEase() each loop; shares the 0-180
clamp + pulse map of setServoAngle. Gait keeps instantaneous writes.

Co-Authored-By: Claude Opus 4.7 (1M context) <noreply@anthropic.com>

* feat(firmware): playClip/tickClip with 500ms return-to-NEUTRAL clip end

One-shot clip player on STATE_ACTION: interpolate clip frames ->
translateToServo -> setJointAngles; at duration end ease all legs to the
neutral stand over 500ms then STATE_IDLE. Pre-empts gait (single motion
owner). Invalid/empty clip ids ignored + logged.

Co-Authored-By: Claude Opus 4.7 (1M context) <noreply@anthropic.com>

* feat(firmware): CMD_PLAY_CLIP=7 {c:id} command + dispatch + API spec

Co-Authored-By: Claude Opus 4.7 (1M context) <noreply@anthropic.com>

* test(firmware): clip parity vs Python _frame_to_servo + placeholder clips_all.h

Generated reference (mirrors gen_ik_reference.py) pins firmware
translateToServo against the exporter's servo conversion within 1 deg.
Placeholder clips_all.h lets the build resolve until the real bundle is
copied in at integration.

Co-Authored-By: Claude Opus 4.7 (1M context) <noreply@anthropic.com>

* chore(firmware): integrate real generated clips_all.h (5 clips)

Replace the placeholder registry with the Blender-generated bundle
(lie down and stand up, one leg lift, tiny wiggle, wave, wiggle).
Firmware builds; all 27 native tests pass (test_clip_interp uses its
own decoupled fixture, unaffected by the swap).

Co-Authored-By: Claude Opus 4.7 (1M context) <noreply@anthropic.com>

* fix(firmware): CMD_CALIBRATE no longer falls through to CMD_MOVE

The break sat inside the 'if keys present' block, so a malformed calibrate
packet (missing id/servo_id/a) skipped the break and fell through into
CMD_MOVE, making the robot start walking. Move the break to the case level
so a malformed calibrate is a harmless no-op. Pre-existing bug, unrelated
to the clip player but found during its review.

Co-Authored-By: Claude Opus 4.7 (1M context) <noreply@anthropic.com>

* docs: clip-player flash/test walkthrough + changelog (Phase 0 + Phase 2)

Add a concise on-robot tutorial (build, flash, connect, play a clip via
{T:7,c:id}, what 'working' looks like) and restructure the changelog into
phase/task-group sections covering the exporter, firmware clip player,
integration, and the fixes found along the way.

Co-Authored-By: Claude Opus 4.7 (1M context) <noreply@anthropic.com>

* docs(plan): Phase-2 on-board clip player implementation plan

The executed plan (W3a exporter + W3b firmware tracks, frozen clips_all.h
contract, grilled decisions). Mirrors the tracked Phase-0 plan.

Co-Authored-By: Claude Opus 4.7 (1M context) <noreply@anthropic.com>

* feat(clip-panel): show active clip's Linear/Bezier preview state

The 'Preview Robot Motion' button flipped interpolation but gave no
indication of which mode the active clip was in. Read the mode live from
the clip's f-curves (new _clip_interpolation_mode helper, same
first-keyframe heuristic the toggle uses) and reflect it on the button:
depressed + 'LINEAR' + linear icon when previewing robot motion, raised +
'BEZIER' + bezier icon when authoring. State is derived, never stored, so
it can't drift from the curves.

Co-Authored-By: Claude Opus 4.7 (1M context) <noreply@anthropic.com>

* feat(clip-panel): configurable ESP IP for exported clip JS

The robot's board IP can change (AP-mode default 192.168.4.1, or a DHCP
lease on a shared network), but the exported .js hardcoded
ws://192.168.4.1:81. Add an 'ESP IP' field (fh_esp_ip scene property,
saved in the .blend) in the Export panel's JS sub-options; to_js() bakes
it into the WebSocket URL and the HOW-TO-RUN comment. Blank falls back to
192.168.4.1; port 81 stays fixed (code/API_SPEC.md). Dry-run is
unaffected (no socket).

Co-Authored-By: Claude Opus 4.7 (1M context) <noreply@anthropic.com>

* chore: gitignore .work/ agent scratch space

Co-Authored-By: Claude Opus 4.7 (1M context) <noreply@anthropic.com>

* fix(firmware): bounds-guard T:4 CMD_CALIBRATE index (G7)

The CMD_CALIBRATE handler indexed LEG_SERVO_CHANNEL[id][servo_id]
(a constexpr uint8_t[4][3]) using raw JSON ints with only a
containsKey check. A malformed T:4 packet (id:7, servo_id:9,
negatives) triggered an out-of-bounds read (UB).

Extract the in-range check to isValidServoIndex() in config.h
(single source of truth next to the array) and reject bad indices
with a [WARN] log + break before the array access. Add a native
Unity test covering id=4, servo_id=3, and negatives.

Co-Authored-By: Claude Opus 4.7 (1M context) <noreply@anthropic.com>

* feat(animation): clamp + warn on out-of-range servo in exporter (G4/G5)

_frame_to_servo() passed out-of-range servo values silently to the
JS/header, relying on the downstream JS/firmware clamp as the only
backstop. Add an explicit clamp to [0,180] plus a per-channel WARNING
(leg, bone, value, frame) so authoring errors surface at export time —
the range companion to the existing FRAME_DELTA_WARN_DEG warning.

This also exposes that the BL shoulder genuinely rails past 180 across
the wave clip (the W6 / round-trip finding), now logged rather than
hidden. Add a test in test_bake_independence.py: a synthetic row driving
BL shoulder over 180 asserts the value clamps to 180 and a WARNING is
printed. Servo parity (in-range) with the firmware is unchanged.

Co-Authored-By: Claude Opus 4.7 (1M context) <noreply@anthropic.com>

* refactor(animation): move scripts to addons/ to align with wiki-setup reorg

Moves files from animation/scripts/ to animation/addons/ to match the
folder split done in feat/wiki-setup (pipeline/ / addons/ / migrations/).
Allows feat/animation-flow-integration to merge into main cleanly before
wiki-setup is ready.

* feat: regularize FL shoulder so servo 90 = outward (Change B) [FLASH HELD]

FL was the lone leg whose shoulder did not map servo 90 to its outward
direction (it used `out.hip = sh`, neutral 75, vs the +135 outward the other
three legs and the convention image use). Regularize it to `90 + (sh - 135)`,
matching FR/BR/BL, so the all-90 calibration pose (Change C) is a symmetric
outward "X" for every leg.

Changed together (firmware + exporter kept byte-identical):
  - motion_math.cpp FL branch: `sh` -> `90 + (sh - 135)`
  - NEUTRAL[FL].sh 75 -> 135; FRONT_LEFT_LEG_HIP_DEFAULT_ANGLE 75 -> 90
  - exporter _frame_to_servo FL branch (animation/addons/fh_clip_panel.py)
  - convention.json neutral_joint_deg.fl[0] 75 -> 135
Tests: test_motion_math FL expectation + a new all-shoulders-outward-is-90
invariant; test_servo_parity FL formula. Also fixed two generators/tests that
still pointed at the pre-move animation/scripts/fh_clip_panel.py path (the file
moved to animation/addons/ in 2f627a1) and regenerated clip_parity_reference.h.
Firmware builds clean; 44/44 native tests pass; servo parity GREEN.

*** DO NOT FLASH until the FL shoulder horn is physically remounted so servo 90
points outward. The code change and the hardware recalibration are inseparable;
flashing without the remount leaves FL ~45 deg off. The exported clip .js/.h
files are still baked with the old FL mapping and must be re-exported before
playing clips on hardware. ***

Co-Authored-By: Claude Opus 4.7 (1M context) <noreply@anthropic.com>

* feat(firmware): reachable flat & stand reference poses via T:2 (Change C)

Expose two reference poses on the existing CMD_STATE (T:2) command:
  s=4 (STATE_REST)  -> relax(): all servos to 90 = flat/spread calibration
                       pose; also clears isInverted (calibration is upright).
  s=5 (STATE_STAND) -> stand(): drive legs to the per-leg NEUTRAL[] table
                       (the gait launch/return pose).

relax() already existed but was dead code (the original all-90 calibration
pose, orphaned when the angle-space gait engine introduced standing-NEUTRAL).
This restores it and adds its standing counterpart. The handler now gates the
wire state through isValidStateCommand() (data.h), widening the accepted range
to include 4/5; out-of-range stays a no-op. Existing s=0..3 behaviour and all
gait/clip paths are unchanged. Documented both states in API_SPEC.md §2.

Native test test_state_command_bounds asserts 0..5 valid, 6/-1/99 rejected.
Firmware builds clean; 35/35 native tests pass.

Co-Authored-By: Claude Opus 4.7 (1M context) <noreply@anthropic.com>

* feat(firmware): smoothstep easing in tickEase (Change 3a)

Replace the linear ramp in Servo::tickEase with a smoothstep ease-in-out
(t*t*(3-2t)) so timed moves accelerate and decelerate instead of starting and
stopping abruptly. Extracted the curve into a pure, host-tested helper
easeFraction() in motion_math.cpp (the Arduino-coupled Servo class isn't
native-buildable, so the math is tested where it can be).

Reaches the target exactly at the end (the t>=dur early-return is unchanged).
Affects the return-to-neutral tail and any setServoAngleTimed move only —
gaits never call tickEase, so gait output is bit-for-bit unchanged.

Native test test_ease_fraction covers endpoints, the exact 0.5 midpoint, the
slow-start/fast-finish quarter points, and the zero-duration case. Firmware
builds clean; 39/39 native tests pass.

Co-Authored-By: Claude Opus 4.7 (1M context) <noreply@anthropic.com>

* feat(firmware): EMA smoothing for clip playback, clip path only (Change 3b)

Apply a per-channel exponential moving average to clip-playback angles inside
tickClip(), between clipPoseAt() and translateToServo(), to take the edge off
jerky keyframe-to-keyframe motion. State is a float[4][3] on SpinalCord seeded
from the clip's first frame on playClip() (so playback starts on the true pose,
no ramp-up). alpha = CLIP_EMA_ALPHA = 0.75 (named, tunable).

Strictly isolated to the clip path: the EMA runs only in CLIP_ACT_APPLY_POSE/
BEGIN_RETURN. Gaits (tickGait/tickTrot/tickYawRotation), calibration, and the
T:4 manual path never touch clipSmoothed_, so gait output is bit-for-bit
unchanged and T:1/T:4/T:5/T:6/T:7 wire behaviour is unchanged. The EMA sits on
pre-invert math-space angles, so it composes correctly with the future unified
invert (Change D), which mirrors at the servo write point.

The smoothing step is the pure helper emaStep() in motion_math.cpp; native test
test_ema_step covers single-step blend, alpha=0 pass-through, convergence to a
held target, and no-overshoot. Firmware builds clean; 43/43 native tests pass.

Co-Authored-By: Claude Opus 4.7 (1M context) <noreply@anthropic.com>

* feat(firmware): unified pitch-only invert at one choke point (Change D)

isInverted was applied only inside the three gait tickers (math-space th=-th,
kn=-kn); clips and the rest ignored it, and invertRobot() wrote a separate
hardcoded inverted pose (which still held FL's pre-Change-B value). Centralize:
all motion now routes its servo triple through SpinalCord::applyServos(), which
mirrors the pitch joints about 90 (thigh, knee; shoulder untouched) when
inverted, via the pure helper applyInvert() in motion_math.

Effects:
  - Gaits: bit-for-bit unchanged. For a pitch servo translateToServo emits
    90±angle, and 180-(90±x) = 90∓x, so the servo-space mirror equals the old
    math-space negation. Proven for all four legs by test_invert_mirror.
  - Clips: now honor invert too (they previously did not) — animations play the
    same flipped or upright, which is the point.
  - invertRobot() (T:6) drops its hardcoded pose table and just toggles the flag
    then re-assumes NEUTRAL through the choke point (mirrored when inverted);
    this also removes the stale hardcoded FL value.
Per-leg flip-axis semantics intentionally out of scope (Marcus): invert is
exactly "hip and knee upside down", nothing more.

EMA (3b) sits on pre-invert math-space

File: code/simulation/generated/facehugger.urdf (robot description, URDF)
Before this commit: robot facehugger, 13 links, 12 joints
Links:
- link base_link: mass 0.565732 -> 1.044732; geometry collision mesh filename=exported_meshes/QuadrupedBody.stl scale=0.001 0.001 0.001; visual mesh filename=exported_meshes/QuadrupedBody.stl scale=0.001 0.001 0.001

Commit message: chore(urdf): regenerate — shell body mass + wider thigh joint limits
Shell body now included in Fusion URDF export: base_link mass 1.045 kg
→ 1.171 kg, inertia tensors updated. Thigh joint limits widened from
±60° (1.047 rad) to ±75° (1.309 rad) to accommodate new animation clips.

Co-Authored-By: Claude Sonnet 4.6 <noreply@anthropic.com>

File: code/simulation/generated/facehugger.urdf (robot description, URDF)
Before this commit: robot facehugger, 13 links, 12 joints
Links:
- link base_link: mass 1.044732 -> 1.170749
Joints:
- joint bl_link2_joint: limit lower=-1.047198 upper=1.047198 effort=2.94 velocity=5.0 -> lower=-1.308997 upper=1.308997 effort=2.94 velocity=5.0
- joint br_link2_joint: limit lower=-1.047198 upper=1.047198 effort=2.94 velocity=5.0 -> lower=-1.308997 upper=1.308997 effort=2.94 velocity=5.0
- joint fl_link2_joint: limit lower=-1.047198 upper=1.047198 effort=2.94 velocity=5.0 -> lower=-1.308997 upper=1.308997 effort=2.94 velocity=5.0
- joint fr_link2_joint: limit lower=-1.047198 upper=1.047198 effort=2.94 velocity=5.0 -> lower=-1.308997 upper=1.308997 effort=2.94 velocity=5.0

Commit message: feat(urdf): add hip+knee servo masses to link1/link3 inertial blocks
link1 (shoulder) and link3 (lower leg) each host one 60g DSS-230MG
servo as a visual-only mesh. Add servo_cfg.mass_kg (0.060 kg) to each
so PyBullet dynamics match the real robot weight distribution.
CoM stays at the structural centroid — adequate for sim fidelity.

Co-Authored-By: Claude Sonnet 4.6 <noreply@anthropic.com>

File: code/simulation/generated/facehugger.urdf (robot description, URDF)
Before this commit: robot facehugger, 13 links, 12 joints
Links:
- link bl_link1: mass 0.149876 -> 0.209876
- link bl_link3: mass 0.127150 -> 0.187150
- link br_link1: mass 0.132968 -> 0.192968
- link br_link3: mass 0.127150 -> 0.187150
- link fl_link1: mass 0.132968 -> 0.192968
- link fl_link3: mass 0.127150 -> 0.187150
- link fr_link1: mass 0.149876 -> 0.209876
- link fr_link3: mass 0.127150 -> 0.187150
