Commit message: fix(urdf): shoulder axis uniform +Z for all legs; remove downstream compensations
All four shoulder servo shafts point in the same direction (+Z body frame).
The link1 bracket STL is mirrored for FR/BL but the servo itself is not, so
the R-side axis negation in generate_urdf.py was wrong. Every downstream layer
had silently compensated: sil_bridge and clip_player multiplied link1 by
LEG_ID_TO_URDF_AXIS_SIGN (FR/BL = −1), and servo_math._LINK1_DELTA_SIGN
cancelled it again on the Blender export path.

Fix the root: remove the shoulder axis negation from generate_urdf.py, drop
the axis factor from link1 in sil_bridge and clip_player, regenerate the URDF.
Hip/knee R-side flips are untouched (those servos ARE physically rotated 180°).

Co-Authored-By: Claude Sonnet 4.6 <noreply@anthropic.com>

File: code/simulation/generated/facehugger.urdf (robot description, URDF)
Before this commit: robot facehugger, 13 links, 12 joints
Joints:
- joint bl_link1_joint: axis 0.0 0.0 -1.0 -> 0.0 0.0 1.0; limit lower=-1.570796 upper=0.907571 effort=2.94 velocity=5.0 -> lower=-0.907571 upper=1.570796 effort=2.94 velocity=5.0
- joint fr_link1_joint: axis 0.0 0.0 -1.0 -> 0.0 0.0 1.0; limit lower=-1.570796 upper=0.907571 effort=2.94 velocity=5.0 -> lower=-0.907571 upper=1.570796 effort=2.94 velocity=5.0

Commit message: refactor(sim/anim): restructure sim packages, modularise urdf_gen, extract animation lib (#108)
* chore(animation): remove stale exported_gaits/, fh_rigged_dancing.blend, migrations/

Three pieces of dead inventory:
- animation/exported_gaits/ — superseded by exported_clips/. The 8
  files inside (lie down and stand up, one leg lift, tiny wiggle,
  wiggle, each as .h + .js) are stale; the firmware's clips_all.h is
  the current source and the .js exports land under
  animation/exported_clips/<clip>/.
- animation/fh_rigged_dancing.blend — historical rig snapshot;
  fh_rigged_latest.blend is the canonical animation library.
- animation/migrations/ — one-shot legacy-name migration was already
  duplicated under animation/scripts/ and deleted there in Phase 0a
  (commit 3dcd104). This drops the directory.

Co-Authored-By: Claude Opus 4.7 (1M context) <noreply@anthropic.com>

* chore: drop stale .gitkeep placeholders (code/notebooks/, lib/)

Both directories no longer exist on disk and have no incoming code or
docs references. The placeholders were anchoring empty directories that
the project never grew into.

Co-Authored-By: Claude Opus 4.7 (1M context) <noreply@anthropic.com>

* chore(doc): move project proposal to repo root as kebab-case

doc/FaceHugger_ProjectProposal.pdf -> FaceHugger-project-proposal.pdf

Visible at the repo root for first-time visitors. Filename style matches
the rest of the wiki/published assets (kebab-case lowercase).

Co-Authored-By: Claude Opus 4.7 (1M context) <noreply@anthropic.com>

* chore: delete docs/CLIP_SHOULDER_CONVENTION.md (fix is in-code)

The doc explained the link1 (shoulder) delta-to-absolute fix as a
narrative postmortem. The fix itself is implemented and the
authoritative explanation now lives in the docstring on
`_link1_delta_to_absolute` in animation/addons/fh_clip_panel.py — the
defect would re-trigger there if anyone reverts the addition of the
per-leg neutral. The clip-shoulder convention overview is covered by
wiki/reference/firmware/kinematics.md.

Rewired the one inbound ref (test_clip_loader.py docstring) to point at
the in-code explanation instead.

Co-Authored-By: Claude Opus 4.7 (1M context) <noreply@anthropic.com>

* chore(animation): refresh fh_rigged_latest.blend

Updated by `facehugger.py blender --rigged --headless` smoke runs
during the simulation reorg phases (the rig builder auto-saves over
this file every run, so the binary contents drift).

Co-Authored-By: Claude Opus 4.7 (1M context) <noreply@anthropic.com>

* cleanup: move doc/ planning docs to .work/, remove historical stubs

doc/animation-pipeline/ was pre-implementation planning; moved to
.work/research/ for maintainer reference. doc/gait-design/ was empty.
doc/torque-analysis/ is already covered by the wiki. Other planning
files moved to .work/context/.

Co-Authored-By: Claude Sonnet 4.6 <noreply@anthropic.com>

* chore(animation): Phase 0a — remove legacy one-shot files

- Delete animation/scripts/RIGGING_PLAN.md: design doc whose implementation
  has shipped (urdf_to_blender_rigged.py); zero inbound references.
- animation/README.md: drop stale `pipeline/` and `migrations/` rows
  (those folders no longer exist), fix `code/simulation/facehugger.py` →
  `code/facehugger.py`, add `lib/` row, list plain-Python tools in scripts/.

Not deleted: animation/scripts/fh_rename_actions.py. Inbound references
in CLAUDE.md, wiki/reference/simulation/scripts-cli.md and two
wiki/_context/ pages mean the delete needs a coordinated wiki/CLAUDE.md
update — out of scope for Phase 0a.

Co-Authored-By: Claude Opus 4.7 (1M context) <noreply@anthropic.com>

* chore(animation): Phase 0a — remove fh_rename_actions.py (legacy one-shot)

Deletes the one-shot legacy Action-rename migration script. Its sibling
copy at animation/migrations/fh_rename_actions.py was already deleted
elsewhere; this finishes the cleanup.

Inbound ref rewires (2):
- CLAUDE.md: drop the mention of fh_rename_actions.py from the
  "animator-facing helpers" paragraph; fh_clip_panel.py is now the
  sole entry there.
- wiki/reference/simulation/scripts-cli.md: remove the "One-shot
  action rename" section and its code block.

The 7 references under wiki/reference/animation/_context/ are
intentionally left in place — those are audit scaffolding that the
user removes manually once the wiki migration is complete (same
policy followed by the Phase 0b wiki migration commits).

Co-Authored-By: Claude Opus 4.7 (1M context) <noreply@anthropic.com>

* chore(cad): update Prusa slicer project files (.3mf)

Body, HipMount, LipoCage, Shell, and leg beds refreshed from latest
Prusa Slicer session. Binary project files only — no geometry changes.

Co-Authored-By: Claude Sonnet 4.6 <noreply@anthropic.com>

* refactor(cad/stls): step 1 — extract config.py

Move ROTATIONS, DEFAULT_UP, LOG_MARKER, VALID_SUBFOLDERS, and SpecEntry
dataclass into a pure-Python config.py with no adsk dependency.
ExportPrintableSTLs.py imports all five and uses VALID_SUBFOLDERS +
SpecEntry in _read_spec so the loop iterates over typed entries.

Co-Authored-By: Claude Sonnet 4.6 <noreply@anthropic.com>

* refactor(cad/urdf): step 1 — extract pure-data modules

Move geometry helpers, STL I/O, landmark resolution, and manifest
builder into config.py, math_utils.py, stl_utils.py, landmark_utils.py,
and manifest.py. Replace inline code in ExportBodiesToURDF.py with
imports from those modules.

Co-Authored-By: Claude Sonnet 4.6 <noreply@anthropic.com>

* refactor(cad/urdf): step 2 — extract verify.py

Move _verify_against_assembly_hierarchy and its _REQUIRED_* constants
into verify.py. Add verify_export_rules_have_physics() to catch missing
physics blocks at export time.

Co-Authored-By: Claude Sonnet 4.6 <noreply@anthropic.com>

* refactor(cad/urdf): step 3 — extract fusion_joints.py

Move collect_joints, _extract_joint, and all joint helpers into
fusion_joints.py. Also moves _find_leg_assembly_R_la there since it
is only used to feed R_la into collect_joints.

Co-Authored-By: Claude Sonnet 4.6 <noreply@anthropic.com>

* refactor(cad/urdf): step 4 — extract fusion_traversal.py

Move traverse, collect_bodies, collect_axes, collect_points,
collect_physics, identity_matrix, mat_multiply, and occ_parent_origin_mm
into fusion_traversal.py.

Co-Authored-By: Claude Sonnet 4.6 <noreply@anthropic.com>

* refactor(cad/urdf): step 5 — extract fusion_stl_export.py

Move export_stls and its helper tree-walk functions into
fusion_stl_export.py. Uses stl_utils.transform_triangles and
landmark_utils for the pure-data operations.

Co-Authored-By: Claude Sonnet 4.6 <noreply@anthropic.com>

* fix(cad): use relative imports inside ExportBodiesToURDF/lib/

Fusion loads lib/ as a package; bare `from config import …` fails because
the package root is not on sys.path. Switch to `from .config import …`
(and similar) so intra-lib imports resolve correctly as relative imports.

Co-Authored-By: Claude Sonnet 4.6 <noreply@anthropic.com>

* refactor(cad): move helper modules into lib/ for both Fusion add-ins

ExportBodiesToURDF and ExportPrintableSTLs now follow a consistent layout:
  - Entry point stays at the add-in root (ExportBodiesToURDF.py / ExportPrintableSTLs.py)
  - All helper modules live in lib/ (config, math_utils, stl_utils, landmark_utils,
    manifest, verify, fusion_traversal, fusion_joints, fusion_stl_export / config, spec_io)
  - Intra-lib imports changed to relative (from .config import ...)
  - Entry-point imports updated to lib.* prefix
  - Tests updated to import from lib.* with add-in root on sys.path
  - .gitignore: suppress __pycache__ inside cad/scripts/ (overridden by the !cad/scripts/** rule)

Co-Authored-By: Claude Sonnet 4.6 <noreply@anthropic.com>

* refactor(cad): ExportBodiesToURDF step 6 — slim entry point to 137 lines

Extracted fmt_tree, fmt_joints, _summarize_joint, fmt_header, fmt_message
into lib/formatters.py (pure dict/string, no adsk). Entry point now
contains only path setup and the run() orchestration function.
303 → 137 lines; formatters.py adds ~160 lines to lib/.

Co-Authored-By: Claude Sonnet 4.6 <noreply@anthropic.com>

* refactor(cad): modularize ExportPrintableSTLs (Steps 3-6)

Step 3: Extract stl_transform.py (rotate_stl_in_place, rotation_for_up_axis);
  add test_stl_transform.py (identity, round-trip, unknown-axis error) and
  test_config.py (orthonormality check for all 6 ROTATIONS matrices).
Step 4: Extract fusion_api.py (iter_occ_tree, find_body, export_body_stl);
  adsk imported only at call-time so module is importable outside Fusion.
Step 5: Deferred (cross-add-in tree-walker dedup).
Step 6: Add DRY_RUN = False toggle to entry point — skip export/rotate when
  set; summary dialog prefixed with [DRY RUN].
Also fix spec_io._is_axis_token to recognise any ±letter as an axis token
so invalid axes like +W raise RuntimeError instead of silently becoming hints.
19/19 host-side tests pass.

Co-Authored-By: Claude Sonnet 4.6 <noreply@anthropic.com>

* refactor(cad): modularize ExportBodiesToURDF into lib/census + lib/stl_export

Merges fusion_traversal.py + fusion_joints.py into lib/census.py (deduped
imports). Moves STL export logic into lib/stl_export.py with ExportOrigin
auto-detection when origin_landmark is absent from a rule. Adds
lib/config_loader.py for YAML-based config loading. Entry point now imports
directly from lib.census and lib.stl_export; shim files removed.

Co-Authored-By: Claude Sonnet 4.6 <noreply@anthropic.com>

* feat(cad): add FaceHuggerExport add-in consolidating URDF + printable STL exports

Co-Authored-By: Claude Sonnet 4.6 <noreply@anthropic.com>

* feat(cad): include Shell body in Fusion URDF export

Re-ran ExportBodiesToURDF with Shell added to EXPORT_RULES combined body.
QuadrupedBody.stl grows 527KB → 2MB (shell mesh included). fusion_export.json
gains Shell occurrence with mass/COM/inertia tensor for physics accuracy.

Co-Authored-By: Claude Sonnet 4.6 <noreply@anthropic.com>

* chore(cad): refresh exports; drop LegMount printable STLs from spec

Re-ran ExportBodiesToURDF and ExportPrintableSTLs after refactor.
Outputs are identical to pre-refactor (STL geometry unchanged; JSON
diff is trailing-newline only). Adds QuadrupedBody.stl to tracking.

Removes LegMountL/R from print_export.txt — the shoulder-mount parts
are already covered by exported_meshes/ for URDF simulation; printable
copies in cad/leg/ are redundant.

Co-Authored-By: Claude Sonnet 4.6 <noreply@anthropic.com>

* chore(cad): remove legacy add-in folders superseded by FaceHuggerExport

ExportBodiesToURDF and ExportPrintableSTLs are now consolidated into
cad/scripts/FaceHuggerExport/ with all tests migrated and passing (70/70).

Co-Authored-By: Claude Sonnet 4.6 <noreply@anthropic.com>

* test(cad): add host-side tests for verify.py (assembly hierarchy + physics)

Co-Authored-By: Claude Sonnet 4.6 <noreply@anthropic.com>

* refactor(fw): step 2 — remove dead Leg::setPose()

Zero call sites confirmed (only the definition in leg.cpp and
declaration in leg.h). Deleted both. Also removed the now-unused
#include "kinematics.h" from leg.cpp since setPose() was the only
caller of legIK().

Co-Authored-By: Claude Sonnet 4.6 <noreply@anthropic.com>

* refactor(fw): step 3 — remove SpinalCord& from initSensors

initSensors(SpinalCord& sc) -> SensorBootResult initSensors().
sensors.h no longer includes spinal_cord.h, severing the brain->
nervous_system header dependency that pulled <Adafruit_PWMServoDriver.h>
into every sensors.h consumer.

main.cpp now acts on the returned SensorBootResult to call
spinalCord.setInverted(true) when boot orientation is inverted.

Co-Authored-By: Claude Sonnet 4.6 <noreply@anthropic.com>

* refactor(fw): step 4 — move input guards into SpinalCord

SpinalCord::setGait() now guards out-of-range GaitType values with an
early return. The equivalent wire-range check in network.cpp is removed.

The outer c >= 0 && c < 256 clip-ID check in network.cpp is removed;
the authoritative guard inside playClip() (id >= FH_CLIP_COUNT) handles
all invalid IDs at one place.

Co-Authored-By: Claude Sonnet 4.6 <noreply@anthropic.com>

* refactor(fw): step 5 — replace leg1..leg4 with legs_[] array

Replace the four named Leg member variables in SpinalCord with
Leg legs_[LEG_COUNT]. All Leg* arr[] = {&leg1,...} temporary
pointer arrays are eliminated; every multi-leg loop now accesses
legs_[i] directly. begin(), snapshot(), relax(), applyCalibration(),
goToNeutral(), easeToNeutral(), flipPoseInPlace(), update(),
tickGait(), tickTrot(), tickYawRotation(), playClip(), and tickClip()
all converted to indexed loops. pio test -e native: 92/92 pass.

Co-Authored-By: Claude Sonnet 4.6 <noreply@anthropic.com>

* refactor(firmware): expose GAITS[] via extern declaration in movements.h (Step 6)

Removes `static` from the GAITS[] definition in spinal_cord.cpp and adds
`extern const GaitParams GAITS[];` to movements.h so any translation unit
that includes movements.h can reference the gait table without pulling in
spinal_cord.cpp. Comment added to both sides marking the split.

Co-Authored-By: Claude Sonnet 4.6 <noreply@anthropic.com>

* firmware: add boot_orientation helpers header for host-testable IMU classification

Pure constexpr/inline helpers (dotUpright, classifyBootOrientation) moved
into a separate header so they can be unit-tested on the native env without
dragging in Wire/MPU stubs. sensors.cpp already uses these via #include.

Co-Authored-By: Claude Sonnet 4.6 <noreply@anthropic.com>

* feat(firmware): add T:12 CMD_STREAM_FRAME — math-space clip streaming with CALIB-at-runtime

Adds a new WebSocket command T:12 that accepts per-frame math-space joint
angles (FR/FL/BR/BL × sh/th/kn) and applies translateToServo + applyInvert
at execution time. This makes exported .js clip files CALIB-agnostic: re-
calibrating the robot no longer requires re-exporting animation clips.

Key additions:
- data.h: CMD_STREAM_FRAME = 12
- config.h: SERVO_DEADBAND_DEG = 0.5f (suppress PWM writes for tiny changes)
- leg.h + leg.cpp: Leg::setServo(servoId, angle) per-joint setter
- spinal_cord.h + spinal_cord.cpp: streamMathFrame() with dirty-flag deadband
- network.cpp: case CMD_STREAM_FRAME parses {fr,fl,br,bl} arrays and dispatches

Co-Authored-By: Claude Sonnet 4.6 <noreply@anthropic.com>

* fix(firmware,sil): correct IMU upright sign convention — +Z when upright

The MPU6050 chip is Z-down: gravity reaction reads +Z (not -Z) when the
robot is upright. Fix the UPRIGHT_REF comment and test vectors in
test_imu_hysteresis, and update the sensors_sil SensorBootResult
signature to match the step-3 refactor (initSensors() → SensorBootResult).

Co-Authored-By: Claude Sonnet 4.6 <noreply@anthropic.com>

* fix(sim): physics P0 — URDF inertia from file, PETG ground-truth config

- Add flags=p.URDF_USE_INERTIA_FROM_FILE to p.loadURDF() in
  _connect_and_setup(). Previously zero flags caused PyBullet to
  silently ignore every <inertial> block in the URDF.
- Add printing: block to facehugger_config.yaml with PETG solid density
  (1.27 g/cm³), per-part infill scale factors (0.151/0.158/0.255 for
  leg links / body+bridges / LiPo cage), and Prusa gcode ground-truth
  masses for all printed parts.
- Fix servo.mass_kg 0.300 → 0.060 (DSS-230MG actual weight).
- Update extra_mass_kg comment: electronics ~0.077 kg (was 0.239 kg
  placeholder); ground-truth estimate ~0.317 kg; value stays at 0.479
  pending full electronics weigh-in.

Co-Authored-By: Claude Sonnet 4.6 <noreply@anthropic.com>

* fix(sim): remove base link mass override — URDF inertia now authoritative

Co-Authored-By: Claude Sonnet 4.6 <noreply@anthropic.com>

* feat(urdf): add hip+knee servo masses to link1/link3 inertial blocks

link1 (shoulder) and link3 (lower leg) each host one 60g DSS-230MG
servo as a visual-only mesh. Add servo_cfg.mass_kg (0.060 kg) to each
so PyBullet dynamics match the real robot weight distribution.
CoM stays at the structural centroid — adequate for sim fidelity.

Co-Authored-By: Claude Sonnet 4.6 <noreply@anthropic.com>

* chore(urdf): regenerate — shell body mass + wider thigh joint limits

Shell body now included in Fusion URDF export: base_link mass 1.045 kg
→ 1.171 kg, inertia tensors updated. Thigh joint limits widened from
±60° (1.047 rad) to ±75° (1.309 rad) to accommodate new animation clips.

Co-Authored-By: Claude Sonnet 4.6 <noreply@anthropic.com>

* refactor(sim): step 1 — move stray files, fix _list_clips

- Move test_package_structure.py to tests/; update SIM_DIR to parent.parent
- Move urdf_gen/verify_export_parity.py to firmware_port/export_parity.py;
  update sys.path.insert to use parents[2] (firmware_port → code/simulation)
- Update test_pipeline_regression.py to search for export_parity.py
- Fix facehugger.py _list_clips() to use firmware_port.clip_loader instead of
  ad-hoc regex

Co-Authored-By: Claude Sonnet 4.6 <noreply@anthropic.com>

* refactor(sim): split helpers.py → math_utils/urdf_io/motor; keep shim

Three focused modules:
- math_utils.py  — _clamp, _wrap_pi, _parse_xyz
- urdf_io.py     — URDF/STL/fusion_export parsing (_load_urdf_joints,
                   _parse_leg_points_from_urdf, _stl_foot_tip_m,
                   _foot_tip_from_fusion)
- motor.py       — PyBullet joint-map + motor helpers (build_joint_map,
                   reset_to_stance, apply_leg_pose, apply_joint_targets)

helpers.py becomes a backwards-compat re-export shim.
kinematics.py and gaits.py updated to import from the new modules.
All 63 sim tests pass.

Co-Authored-By: Claude Sonnet 4.6 <noreply@anthropic.com>

* refactor(sim): extract pybullet_sim/scene.py (connect_and_setup, settle, print_banner)

Move PyBullet scene lifecycle out of gaits.py into a dedicated scene.py:
- connect_and_setup / settle / print_banner (public names, no leading _)
- physics constants moved here (FOOT_LATERAL_FRICTION, etc.)

gaits.py: import from scene under the original private-name aliases so all
call sites are unchanged (no churn). Removes pybullet_data / apply_leg_pose /
build_joint_map / reset_to_stance imports no longer needed in gaits.

ws_sim.py: now imports connect_and_setup from pybullet_sim.scene directly
instead of reaching into the private _connect_and_setup in gaits.

Co-Authored-By: Claude Sonnet 4.6 <noreply@anthropic.com>

* refactor(sim): extract pybullet_sim/runner.py (run_stand/gait/clip + step hooks)

Move run loops and step-monitor helpers out of gaits.py into runner.py:
- run_stand, run_clip, _run_clip_sil, _run_gait_sil, run_gait
- setup_step_hook, _make_step_monitor, _finalize_log

gaits.py now contains only gait IK math: GAITS, foot_target,
gait_joint_targets, _precompute_cycle, _draw_overlay, _body_height_for_gait.
Backward-compat re-exports added so existing gaits.py importers still work.

simulate.py: updated to import run_* from runner directly.

Co-Authored-By: Claude Sonnet 4.6 <noreply@anthropic.com>

* refactor(sim): Steps 5-7 — split sil_bridge, add paths.py, remove shims

Step 5: Split firmware_sil/sil_bridge.py into focused sub-modules:
  - build.py   — CMake staleness check + load_fh_sim
  - imu.py     — PyBullet→firmware IMU hysteresis + pitch/roll
  - telemetry.py — torque colors + per-step telemetry frame
  - trace.py   — deterministic clip/gait traces for regression testing
  sil_bridge.py becomes the orchestration layer re-exporting all public names;
  63 tests pass.

Step 6: Extract path constants from constants.py into pybullet_sim/paths.py
  (single source of truth for SIM_ROOT, GENERATED_DIR, URDF_PATH, etc.).
  constants.py re-exports them for backward compat; keeps TIMESTEP/STANCE_DEG.

Step 7: Remove helpers.py backwards-compat shim, firmware_port/gait_interpreter.py
  stub, and terrain_report.md orphan. Update two test files + test_package_structure
  to import build_joint_map from motor directly.

Also add ExportBodiesToURDF host-side tests (Step 7 for the Fusion add-in):
  test_math_utils, test_stl_utils, test_landmark_utils, test_manifest.
  test_verify is in progress.

Co-Authored-By: Claud

File: code/simulation/generated/facehugger.urdf (robot description, URDF)
Before this commit: robot facehugger, 13 links, 12 joints
Links:
- link base_link: mass 1.044732 -> 1.170749
- link bl_link1: mass 0.149876 -> 0.209876
- link bl_link3: mass 0.127150 -> 0.187150
- link br_link1: mass 0.132968 -> 0.192968
- link br_link3: mass 0.127150 -> 0.187150
- link fl_link1: mass 0.132968 -> 0.192968
- link fl_link3: mass 0.127150 -> 0.187150
- link fr_link1: mass 0.149876 -> 0.209876
- link fr_link3: mass 0.127150 -> 0.187150
Joints:
- joint bl_link2_joint: limit lower=-1.047198 upper=1.047198 effort=2.94 velocity=5.0 -> lower=-1.308997 upper=1.308997 effort=2.94 velocity=5.0
- joint br_link2_joint: limit lower=-1.047198 upper=1.047198 effort=2.94 velocity=5.0 -> lower=-1.308997 upper=1.308997 effort=2.94 velocity=5.0
- joint fl_link2_joint: limit lower=-1.047198 upper=1.047198 effort=2.94 velocity=5.0 -> lower=-1.308997 upper=1.308997 effort=2.94 velocity=5.0
- joint fr_link2_joint: limit lower=-1.047198 upper=1.047198 effort=2.94 velocity=5.0 -> lower=-1.308997 upper=1.308997 effort=2.94 velocity=5.0
