Commit message: feat(urdf): per-body-side asymmetric shoulder limits
Aligns the URDF and the Blender rig with the firmware safety net
(SHOULDER_THETA_NARROW_DEG / SHOULDER_THETA_WIDE_DEG in config.h,
slice 1). The shoulder axis stays uniform +Z across all four legs
(dc97133); only the URDF <limit> window is mirrored per body side:

  LEFT  body (FL, BL):  θ ∈ [-52°, +90°]   (URDF tight inward, loose outward)
  RIGHT body (FR, BR):  θ ∈ [-90°, +52°]   (mirror)

The mirror picks the loose-θ direction to be the physically OUTWARD
direction for each leg — the same window the firmware's
enforceShoulderLimits clamps to and the Blender LIMIT_ROTATION + IK
Z-limit constraints inherit from the URDF. Animator now gets hard IK
clamping in Blender that matches what firmware will allow at runtime.

The body-side determination uses the leg_id suffix ('r' / 'l') rather
than the facehugger_config.yaml `side` field, because that field tracks
bracket pairing (L-bracket = FL+BR, R-bracket = FR+BL) used for the
hip/knee axis flip — NOT body side.

Rebuilt fh_rigged_latest.blend so the Blender rig's per-shoulder
LIMIT_ROTATION + use_ik_limit_z reflect the new asymmetric envelope.

Co-Authored-By: Claude Opus 4.7 <noreply@anthropic.com>

File: code/simulation/generated/facehugger.urdf (robot description, URDF)
Before this commit: robot facehugger, 13 links, 12 joints
Joints:
- joint br_link1_joint: limit lower=-0.907571 upper=1.570796 effort=2.94 velocity=5.0 -> lower=-1.570796 upper=0.907571 effort=2.94 velocity=5.0
- joint fr_link1_joint: limit lower=-0.907571 upper=1.570796 effort=2.94 velocity=5.0 -> lower=-1.570796 upper=0.907571 effort=2.94 velocity=5.0

Commit message: feat: shoulder-limit + inter-leg alignment across URDF, rig, firmware, lint; CALIB   decoupling (#111)
* feat(clips): export new clips, sync firmware and app manifests

Adds twerk, body-wave, imbalance-flip, roll-ish; updates dog-walk,
one-leg-lift, and several existing clips with tuned keyframes.
Syncs clips_all.h (firmware) and clips_extra.json (app). Adds AGENTS.md
for agentic session context.

Co-Authored-By: Claude Sonnet 4.6 <noreply@anthropic.com>

* firmware: add boot_orientation helpers header for host-testable IMU classification

Pure constexpr/inline helpers (dotUpright, classifyBootOrientation) moved
into a separate header so they can be unit-tested on the native env without
dragging in Wire/MPU stubs. sensors.cpp already uses these via #include.

Co-Authored-By: Claude Sonnet 4.6 <noreply@anthropic.com>

* wiki: reformat team page, clean up social links

Co-Authored-By: Claude Sonnet 4.6 <noreply@anthropic.com>

* cleanup: move doc/ planning docs to .work/, remove historical stubs

doc/animation-pipeline/ was pre-implementation planning; moved to
.work/research/ for maintainer reference. doc/gait-design/ was empty.
doc/torque-analysis/ is already covered by the wiki. Other planning
files moved to .work/context/.

Co-Authored-By: Claude Sonnet 4.6 <noreply@anthropic.com>

* wiki: fix factual errors, update API reference, remove em dashes

Factual fixes:
- motion-engine.md: FL shoulder NEUTRAL corrected 75 -> 135 (post-Change-B)
- assembly.md: servo channel table replaced with correct config.h mapping
  (BL=0-2, BR=4-6, FR=8-10, FL=12-14; old table had FR at ch 0)
- wiring.md: schematic SVG now renders (image tag was inside backticks)
- assembly.md: broken internal link fixed (image syntax -> proper link)

API reference (api.md) updated to current protocol:
- T:2: add REST (4) and STAND (5) states, document optional dur_ms easing
- T:6: replace retired CMD_ACTION_SELECTION with CMD_SET_AUTO_INVERT
- T:7: update clip list to 10 current clips, add loop field
- T:8/T:9/T:11: new commands (List Clips, Set Invert, Set Clip Smoothing)
- T:10: add pitch_deg, roll_deg, upside_down, auto_invert_enabled fields

Style: ~65 em dashes replaced with hyphens across 12 wiki files

Co-Authored-By: Claude Sonnet 4.6 <noreply@anthropic.com>

* wiki: remove internal change/convention labels, rewrite as current-state facts

Internal development labels ('Change B', 'change B') replaced with
plain descriptions of the current hardware and software state. The
wiki is public documentation; historical change markers are not
meaningful to builders or extenders.

Co-Authored-By: Claude Sonnet 4.6 <noreply@anthropic.com>

* fix(sim): physics P0 — URDF inertia from file, PETG ground-truth config

- Add flags=p.URDF_USE_INERTIA_FROM_FILE to p.loadURDF() in
  _connect_and_setup(). Previously zero flags caused PyBullet to
  silently ignore every <inertial> block in the URDF.
- Add printing: block to facehugger_config.yaml with PETG solid density
  (1.27 g/cm³), per-part infill scale factors (0.151/0.158/0.255 for
  leg links / body+bridges / LiPo cage), and Prusa gcode ground-truth
  masses for all printed parts.
- Fix servo.mass_kg 0.300 → 0.060 (DSS-230MG actual weight).
- Update extra_mass_kg comment: electronics ~0.077 kg (was 0.239 kg
  placeholder); ground-truth estimate ~0.317 kg; value stays at 0.479
  pending full electronics weigh-in.

Co-Authored-By: Claude Sonnet 4.6 <noreply@anthropic.com>

* refactor(cad/stls): step 1 — extract config.py

Move ROTATIONS, DEFAULT_UP, LOG_MARKER, VALID_SUBFOLDERS, and SpecEntry
dataclass into a pure-Python config.py with no adsk dependency.
ExportPrintableSTLs.py imports all five and uses VALID_SUBFOLDERS +
SpecEntry in _read_spec so the loop iterates over typed entries.

Co-Authored-By: Claude Sonnet 4.6 <noreply@anthropic.com>

* refactor(fw): step 5 — replace leg1..leg4 with legs_[] array

Replace the four named Leg member variables in SpinalCord with
Leg legs_[LEG_COUNT]. All Leg* arr[] = {&leg1,...} temporary
pointer arrays are eliminated; every multi-leg loop now accesses
legs_[i] directly. begin(), snapshot(), relax(), applyCalibration(),
goToNeutral(), easeToNeutral(), flipPoseInPlace(), update(),
tickGait(), tickTrot(), tickYawRotation(), playClip(), and tickClip()
all converted to indexed loops. pio test -e native: 91/93 pass
(pre-existing imu_hysteresis failure unchanged).

Co-Authored-By: Claude Sonnet 4.6 <noreply@anthropic.com>

* refactor(cad/urdf): step 1 — extract pure-data modules

Move geometry helpers, STL I/O, landmark resolution, and manifest
builder into config.py, math_utils.py, stl_utils.py, landmark_utils.py,
and manifest.py. Replace inline code in ExportBodiesToURDF.py with
imports from those modules.

Co-Authored-By: Claude Sonnet 4.6 <noreply@anthropic.com>

* refactor(cad/urdf): step 2 — extract verify.py

Move _verify_against_assembly_hierarchy and its _REQUIRED_* constants
into verify.py. Add verify_export_rules_have_physics() to catch missing
physics blocks at export time.

Co-Authored-By: Claude Sonnet 4.6 <noreply@anthropic.com>

* refactor(cad/urdf): step 3 — extract fusion_joints.py

Move collect_joints, _extract_joint, and all joint helpers into
fusion_joints.py. Also moves _find_leg_assembly_R_la there since it
is only used to feed R_la into collect_joints.

Co-Authored-By: Claude Sonnet 4.6 <noreply@anthropic.com>

* refactor(cad/urdf): step 4 — extract fusion_traversal.py

Move traverse, collect_bodies, collect_axes, collect_points,
collect_physics, identity_matrix, mat_multiply, and occ_parent_origin_mm
into fusion_traversal.py.

Co-Authored-By: Claude Sonnet 4.6 <noreply@anthropic.com>

* refactor(cad/urdf): step 5 — extract fusion_stl_export.py

Move export_stls and its helper tree-walk functions into
fusion_stl_export.py. Uses stl_utils.transform_triangles and
landmark_utils for the pure-data operations.

Co-Authored-By: Claude Sonnet 4.6 <noreply@anthropic.com>

* refactor(fw): step 2 — remove dead Leg::setPose()

Zero call sites confirmed (only the definition in leg.cpp and
declaration in leg.h). Deleted both. Also removed the now-unused
#include "kinematics.h" from leg.cpp since setPose() was the only
caller of legIK().

Co-Authored-By: Claude Sonnet 4.6 <noreply@anthropic.com>

* refactor(fw): step 3 — remove SpinalCord& from initSensors

initSensors(SpinalCord& sc) -> SensorBootResult initSensors().
sensors.h no longer includes spinal_cord.h, severing the brain->
nervous_system header dependency that pulled <Adafruit_PWMServoDriver.h>
into every sensors.h consumer.

main.cpp now acts on the returned SensorBootResult to call
spinalCord.setInverted(true) when boot orientation is inverted.

Co-Authored-By: Claude Sonnet 4.6 <noreply@anthropic.com>

* refactor(fw): step 4 — move input guards into SpinalCord

SpinalCord::setGait() now guards out-of-range GaitType values with an
early return. The equivalent wire-range check in network.cpp is removed.

The outer c >= 0 && c < 256 clip-ID check in network.cpp is removed;
the authoritative guard inside playClip() (id >= FH_CLIP_COUNT) handles
all invalid IDs at one place.

Co-Authored-By: Claude Sonnet 4.6 <noreply@anthropic.com>

* refactor(fw): step 5 — replace leg1..leg4 with legs_[] array

Replace the four named Leg member variables in SpinalCord with
Leg legs_[LEG_COUNT]. All Leg* arr[] = {&leg1,...} temporary
pointer arrays are eliminated; every multi-leg loop now accesses
legs_[i] directly. begin(), snapshot(), relax(), applyCalibration(),
goToNeutral(), easeToNeutral(), flipPoseInPlace(), update(),
tickGait(), tickTrot(), tickYawRotation(), playClip(), and tickClip()
all converted to indexed loops. pio test -e native: 92/92 pass.

Co-Authored-By: Claude Sonnet 4.6 <noreply@anthropic.com>

* fix(sim): remove base link mass override — URDF inertia now authoritative

Co-Authored-By: Claude Sonnet 4.6 <noreply@anthropic.com>

* refactor(sim): step 1 — move stray files, fix _list_clips

- Move test_package_structure.py to tests/; update SIM_DIR to parent.parent
- Move urdf_gen/verify_export_parity.py to firmware_port/export_parity.py;
  update sys.path.insert to use parents[2] (firmware_port → code/simulation)
- Update test_pipeline_regression.py to search for export_parity.py
- Fix facehugger.py _list_clips() to use firmware_port.clip_loader instead of
  ad-hoc regex

Co-Authored-By: Claude Sonnet 4.6 <noreply@anthropic.com>

* refactor(anim): step 1 — consolidate bpy_stub.py into animation/lib/

Create animation/lib/bpy_stub.py with a single install() function that
merges the three near-identical _stub_bpy() implementations. Update
test_servo_parity.py and check_export_consistency.py to call
bpy_stub.install(); delete their local stub copies. Add animation/lib/
to version control (exempted from the root .gitignore lib/ rule).

Co-Authored-By: Claude Sonnet 4.6 <noreply@anthropic.com>

* fix(animation): add missing bpy_stub import in check_export_consistency + test_servo_parity

Both scripts were calling bpy_stub.install() without importing the module,
causing NameError at runtime after the lib consolidation cherry-pick.

Co-Authored-By: Claude Sonnet 4.6 <noreply@anthropic.com>

* chore(cad): update Prusa slicer project files (.3mf)

Body, HipMount, LipoCage, Shell, and leg beds refreshed from latest
Prusa Slicer session. Binary project files only — no geometry changes.

Co-Authored-By: Claude Sonnet 4.6 <noreply@anthropic.com>

* feat(cad): include Shell body in Fusion URDF export

Re-ran ExportBodiesToURDF with Shell added to EXPORT_RULES combined body.
QuadrupedBody.stl grows 527KB → 2MB (shell mesh included). fusion_export.json
gains Shell occurrence with mass/COM/inertia tensor for physics accuracy.

Co-Authored-By: Claude Sonnet 4.6 <noreply@anthropic.com>

* refactor(cad): move helper modules into lib/ for both Fusion add-ins

ExportBodiesToURDF and ExportPrintableSTLs now follow a consistent layout:
  - Entry point stays at the add-in root (ExportBodiesToURDF.py / ExportPrintableSTLs.py)
  - All helper modules live in lib/ (config, math_utils, stl_utils, landmark_utils,
    manifest, verify, fusion_traversal, fusion_joints, fusion_stl_export / config, spec_io)
  - Intra-lib imports changed to relative (from .config import ...)
  - Entry-point imports updated to lib.* prefix
  - Tests updated to import from lib.* with add-in root on sys.path
  - .gitignore: suppress __pycache__ inside cad/scripts/ (overridden by the !cad/scripts/** rule)

Co-Authored-By: Claude Sonnet 4.6 <noreply@anthropic.com>

* refactor(cad): ExportBodiesToURDF step 6 — slim entry point to 137 lines

Extracted fmt_tree, fmt_joints, _summarize_joint, fmt_header, fmt_message
into lib/formatters.py (pure dict/string, no adsk). Entry point now
contains only path setup and the run() orchestration function.
303 → 137 lines; formatters.py adds ~160 lines to lib/.

Co-Authored-By: Claude Sonnet 4.6 <noreply@anthropic.com>

* feat(firmware): add T:12 CMD_STREAM_FRAME — math-space clip streaming with CALIB-at-runtime

Adds a new WebSocket command T:12 that accepts per-frame math-space joint
angles (FR/FL/BR/BL × sh/th/kn) and applies translateToServo + applyInvert
at execution time. This makes exported .js clip files CALIB-agnostic: re-
calibrating the robot no longer requires re-exporting animation clips.

Key additions:
- data.h: CMD_STREAM_FRAME = 12
- config.h: SERVO_DEADBAND_DEG = 0.5f (suppress PWM writes for tiny changes)
- leg.h + leg.cpp: Leg::setServo(servoId, angle) per-joint setter
- spinal_cord.h + spinal_cord.cpp: streamMathFrame() with dirty-flag deadband
- network.cpp: case CMD_STREAM_FRAME parses {fr,fl,br,bl} arrays and dispatches

Co-Authored-By: Claude Sonnet 4.6 <noreply@anthropic.com>

* docs(api): document T:12 CMD_STREAM_FRAME — math-space clip streaming

Adds the T:12 specification to API_SPEC.md: per-frame math-space joint angles
(fr/fl/br/bl × [sh,th,kn]), dirty-flag deadband, invert-aware behaviour, and
the motivation for switching from T:4 servo-space to T:12 math-space so clip
files are CALIB-agnostic.

Co-Authored-By: Claude Sonnet 4.6 <noreply@anthropic.com>

* refactor(animation): to_js() outputs T:12 math-space frames (CALIB-agnostic)

Switches the browser-console clip export from per-joint T:4 servo-space
commands to a single T:12 math-space frame per tick. Key changes:
- Use _scale_from_neutral() instead of _frame_to_servo() for clip data
- Format angles as 4dp floats (not rounded integers)
- playFrame() sends one {T:12, fr, fl, br, bl} message per frame
- Remove LEG_IDS, clamp helper, and _last delta-cache from JS template
- Update header comments to reflect T:12 wire shape

Clip files exported with this version are CALIB-agnostic: re-calibrating
the robot does not require re-exporting animations.

Co-Authored-By: Claude Sonnet 4.6 <noreply@anthropic.com>

* chore(clips): regenerate all .js clip files as T:12 math-space streams

Replaces per-joint T:4 servo-angle commands with single T:12 math-space
frame messages. Angles sourced directly from clips_all.h (pre-scaled
math-space, already scale-from-NEUTRAL applied); firmware applies
translateToServo + CALIB at runtime.

All 10 clips updated: Twerk, body wave, dancing, dancing up and down,
dog walk, imbalance flip, lie down and stand up, one leg lift, roll-ish,
wave, wiggle.

Co-Authored-By: Claude Sonnet 4.6 <noreply@anthropic.com>

* refactor(sim): simplify export_parity.py for T:12 math-space identity check

With T:12, .js clip files carry math-space angles directly (no CALIB pre-
applied). The parity check is now a simple identity assertion: .js values
must match clips_all.h within 0.001° (4dp rounding tolerance).

Removes: _clamp_0_180, _sim_servo_js_equiv, translate_to_servo import.
Updates: _parse_js_frames parses floats; verify_clip does direct comparison.
All 10 clips pass (10/10 PASS).

Co-Authored-By: Claude Sonnet 4.6 <noreply@anthropic.com>

* fix(firmware,sil): correct IMU upright sign convention — +Z when upright

The MPU6050 chip is Z-down: gravity reaction reads +Z (not -Z) when the
robot is upright. Fix the UPRIGHT_REF comment and test vectors in
test_imu_hysteresis, and update the sensors_sil SensorBootResult
signature to match the step-3 refactor (initSensors() → SensorBootResult).

Co-Authored-By: Claude Sonnet 4.6 <noreply@anthropic.com>

* fix(sim): use CALIB-relative invert mirror in test_sil_invert

applyInvert() mirrors about (2*CALIB - s) not (180 - s), so the test's
_neutral_servo_angles(inverted=True) was wrong. Updated to import
CALIB_THIGH / CALIB_KNEE and apply the same formula.

Co-Authored-By: Claude Sonnet 4.6 <noreply@anthropic.com>

* chore(urdf): regenerate — shell body mass + wider thigh joint limits

Shell body now included in Fusion URDF export: base_link mass 1.045 kg
→ 1.171 kg, inertia tensors updated. Thigh joint limits widened from
±60° (1.047 rad) to ±75° (1.309 rad) to accommodate new animation clips.

Co-Authored-By: Claude Sonnet 4.6 <noreply@anthropic.com>

* fix(cad): use relative imports inside ExportBodiesToURDF/lib/

Fusion loads lib/ as a package; bare `from config import …` fails because
the package root is not on sys.path. Switch to `from .config import …`
(and similar) so intra-lib imports resolve correctly as relative imports.

Co-Authored-By: Claude Sonnet 4.6 <noreply@anthropic.com>

* fix(sil): reset shared SpinalCord state in FirmwareControl constructor

spinalCord is a module-level global. FirmwareControl() called begin() which
resets isInverted but not clipEmaAlpha_ (0.75f boot default) or
autoInvertEnabled_ (true). test_sil_clip_smoothing set alpha=0.95 and
leaked it into subsequent golden-trace tests, causing 1-degree diffs.

Also update CLIP_ID in test_sil_clip_loop from 2 → 6: "one leg lift"
shifted when the 4 new clips (Twerk, body wave, dog walk, roll-ish) were
prepended to FH_CLIPS[].

Co-Authored-By: Claude Sonnet 4.6 <noreply@anthropic.com>

* chore(sil): regenerate golden traces for T:12 clip format + 4 new clips

All 10 clips now stream T:12 math-space frames (CALIB-agnostic). Adds
4 new golden files: twerk, body_wave, dog_walk, roll_ish. Regenerated
with `python -m firmware_sil.gen_golden` after all clip .js files were
re-exported.

Co-Authored-By: Claude Sonnet 4.6 <noreply@anthropic.com>

* fix(sim): test_sil_clip_loop looks up clip by name, skips if absent

Hardcoded CLIP_ID was fragile against clip list reorders. Now uses T:8 to
find "one leg lift" by name and reads its duration directly. If the clip is
removed from the firmware build, the test skips with a warning instead of
failing — the clip library is still in flux.

Co-Authored-By: Claude Sonnet 4.6 <noreply@anthropic.com>

* refactor(sil): rename golden→reference_clips, expose update-reference-clips CLI

- firmware_sil/golden/ → firmware_sil/reference_clips/
- gen_golden.py → gen_references.py
- facehugger.py: add `update-reference-clips` subcommand
- facehugger_config.yaml: add reference_clips: list (wiggle, dog walk,
  wave, lie down and stand up) — CI hard-fails only for these; other
  clips warn on mismatch so active authoring doesn't break the suite
- test_sil_clip_suite.py: load required names from config, two-tier
  pass/warn behaviour; regenerate command in docstring
- README.md, sil_bridge.py: update references

Co-Authored-By: Claude Sonnet 4.6 <noreply@anthropic.com>

* feat(urdf): add hip+knee servo masses to link1/link3 inertial blocks

link1 (shoulder) and link3 (lower leg) each host one 60g DSS-230MG
servo as a visual-only mesh. Add servo_cfg.mass_kg (0.060 kg) to each
so PyBullet dynamics match the real robot weight distribution.
CoM stays at the structural centroid — adequate for sim fidelity.

Co-Authored-By: Claude Sonnet 4.6 <noreply@anthropic.com>

* refactor(sim): split helpers.py → math_utils/urdf_io/motor; keep shim

Three focused modules:
- math_utils.py  — _clamp, _wrap_pi, _parse_xyz
- urdf_io.py     — URDF/STL/fusion_export parsing (_load_urdf_joints,
                   _parse_leg_points_from_urdf, _stl_foot_tip_m,
                   _foot_tip_from_fusion)
- motor.py       — PyBullet joint-map + motor helpers (build_joint_map,
                   reset_to_stance, apply_leg_pose, apply_joint_targets)

helpers.py becomes a backwards-compat re-export shim.
kinematics.py and gaits.py updated to import from the new modules.
All 63 sim tests pass.

Co-Authored-By: Claude Sonnet 4.6 <noreply@anthropic.com>

* refactor(sim): extract pybullet_sim/scene.py (connect_and_setup, settle, print_banner)

Move PyBullet scene lifecycle out of gaits.py into a dedicated scene.py:
- connect_and_setup / settle / print_banner (public names, no leading _)
- physics constants moved here (FOOT_LATERAL_FRICTION, etc.)

gaits.py: import from scene under the original private-name aliases so all
call sites are unchanged (no churn). Removes pybullet_data / apply_leg_pose /
build_joint_map / reset_to_stance imports no longer needed in gaits.

ws_sim.py: now imports connect_and_setup from pybullet_sim.scene directly
instead of reaching into the private _connect_and_setup in gaits.

Co-Authored-By: Claude Sonnet 4.6 <noreply@anthropic.com>

* refactor(sim): extract pybullet_sim/runner.py (run_stand/gait/clip + step hooks)

Move run loops and step-monitor helpers out of gaits.py into runner.py:
- run_stand, run_clip, _run_clip_sil, _run_gait_sil, run_gait
- setup_step_hook, _make_step_monitor, _finalize_log

gaits.py now contains only gait IK math: GAITS, foot_target,
gait_joint_targets, _precompute_cycle, _draw_overlay, _body_height_for_gait.
Backward-compat re-exports added so existing gaits.py importers still work.

simulate.py: updated to import run_* from runner directly.

Co-Authored-By: Claude Sonnet 4.6 <noreply@anthropic.com>

* refactor(sim): Steps 5-7 — split sil_bridge, add paths.py, remove shims

Step 5: Split firmware_sil/sil_bridge.py into focused sub-modules:
  - build.py   — CMake staleness check + load_fh_sim
  - imu.py     — PyBullet→firmware IMU hysteresis + pitch/roll
  - telemetry.py — torque

File: code/simulation/generated/facehugger.urdf (robot description, URDF)
Before this commit: robot facehugger, 13 links, 12 joints
Joints:
- joint bl_link1_joint: axis 0.0 0.0 -1.0 -> 0.0 0.0 1.0; limit lower=-1.570796 upper=0.907571 effort=2.94 velocity=5.0 -> lower=-0.907571 upper=1.570796 effort=2.94 velocity=5.0
- joint br_link1_joint: limit lower=-0.907571 upper=1.570796 effort=2.94 velocity=5.0 -> lower=-1.570796 upper=0.907571 effort=2.94 velocity=5.0
- joint fr_link1_joint: axis 0.0 0.0 -1.0 -> 0.0 0.0 1.0
