Commit message: feat(cad): regenerate export — updated component names, Link2/3 geometry refresh, mass/COM update

File: code/simulation/generated/facehugger.urdf (robot description, URDF)
Before this commit: robot facehugger, 13 links, 12 joints
Links:
- link base_link: geometry collision mesh filename=exported_meshes/QuadrupedBody.stl scale=0.001 0.001 0.001; visual mesh filename=exported_meshes/QuadrupedBody.stl scale=0.001 0.001 0.001
- link bl_link1: mass 0.134355 -> 0.149876
- link bl_link2: mass 0.152739 -> 0.141725
- link bl_link3: mass 0.136030 -> 0.131103
- link br_link1: mass 0.134355 -> 0.132968
- link br_link2: mass 0.152739 -> 0.141725
- link br_link3: mass 0.136030 -> 0.131103
- link fl_link1: mass 0.134355 -> 0.132968
- link fl_link2: mass 0.152739 -> 0.141725
- link fl_link3: mass 0.136030 -> 0.131103
- link fr_link1: mass 0.134355 -> 0.149876
- link fr_link2: mass 0.152739 -> 0.141725
- link fr_link3: mass 0.136030 -> 0.131103
Joints:
- joint bl_link2_joint: origin xyz=0.055920 0.022595 -0.031598 rpy=0 0 0.0 -> xyz=0.046920 0.022395 -0.031598 rpy=0 0 0.0
- joint bl_link3_joint: origin xyz=0.060700 0.000005 0.000000 rpy=0 0 0.0 -> xyz=0.059700 0.000205 0.000000 rpy=0 0 0.0
- joint br_link2_joint: origin xyz=-0.055920 0.022595 -0.031598 rpy=0 0 0.0 -> xyz=-0.046920 0.022395 -0.031598 rpy=0 0 0.0
- joint br_link3_joint: origin xyz=-0.060700 0.000005 0.000000 rpy=0 0 0.0 -> xyz=-0.059700 0.000205 0.000000 rpy=0 0 0.0
- joint fl_link2_joint: origin xyz=-0.055920 0.022595 -0.031598 rpy=0 0 0.0 -> xyz=-0.046920 0.022395 -0.031598 rpy=0 0 0.0
- joint fl_link3_joint: origin xyz=-0.060700 0.000005 0.000000 rpy=0 0 0.0 -> xyz=-0.059700 0.000205 0.000000 rpy=0 0 0.0
- joint fr_link2_joint: origin xyz=0.055920 0.022595 -0.031598 rpy=0 0 0.0 -> xyz=0.046920 0.022395 -0.031598 rpy=0 0 0.0
- joint fr_link3_joint: origin xyz=0.060700 0.000005 0.000000 rpy=0 0 0.0 -> xyz=0.059700 0.000205 0.000000 rpy=0 0 0.0

Commit message: feat: replace STL collision with analytic primitives on leg links
- urdf_writer.py: add CollisionPrimitive dataclass (sphere/box) and
  collision_override parameter to link(). When override is provided,
  emit analytic geometry instead of STL mesh for collision.
- generate_urdf.py: compute foot tip once in _build_state(), store in
  _GenState. Emit sphere (r=5mm) at foot tip for link3, boxes (15mm
  cross-section) along bone direction for link1 and link2.
- R-pair link3 foot tip applies Ry(pi) mirror via (-x, y, -z) transform
  to match the mesh_rpy flip on the visual.
- base_link keeps STL collision (chassis shape matters for flip/drop).
- Regenerated facehugger.urdf.

All 60 urdf/foot_tip/joint tests pass. URDF loads in PyBullet DIRECT.

File: code/simulation/generated/facehugger.urdf (robot description, URDF)
Before this commit: robot facehugger, 13 links, 12 joints
Links:
- link bl_link1: geometry collision box size=0.060840 0.015000 0.015000; visual mesh filename=exported_meshes/leg_shoulder_R.stl scale=0.001 0.001 0.001
- link bl_link2: geometry collision box size=0.074700 0.015000 0.015000; visual mesh filename=exported_meshes/leg_upper.stl scale=0.001 0.001 0.001
- link bl_link3: geometry collision sphere radius=0.005; visual mesh filename=exported_meshes/leg_lower.stl scale=0.001 0.001 0.001
- link br_link1: geometry collision box size=0.060840 0.015000 0.015000; visual mesh filename=exported_meshes/leg_shoulder_L.stl scale=0.001 0.001 0.001
- link br_link2: geometry collision box size=0.074700 0.015000 0.015000; visual mesh filename=exported_meshes/leg_upper.stl scale=0.001 0.001 0.001
- link br_link3: geometry collision sphere radius=0.005; visual mesh filename=exported_meshes/leg_lower.stl scale=0.001 0.001 0.001
- link fl_link1: geometry collision box size=0.060840 0.015000 0.015000; visual mesh filename=exported_meshes/leg_shoulder_L.stl scale=0.001 0.001 0.001
- link fl_link2: geometry collision box size=0.074700 0.015000 0.015000; visual mesh filename=exported_meshes/leg_upper.stl scale=0.001 0.001 0.001
- link fl_link3: geometry collision sphere radius=0.005; visual mesh filename=exported_meshes/leg_lower.stl scale=0.001 0.001 0.001
- link fr_link1: geometry collision box size=0.060840 0.015000 0.015000; visual mesh filename=exported_meshes/leg_shoulder_R.stl scale=0.001 0.001 0.001
- link fr_link2: geometry collision box size=0.074700 0.015000 0.015000; visual mesh filename=exported_meshes/leg_upper.stl scale=0.001 0.001 0.001
- link fr_link3: geometry collision sphere radius=0.005; visual mesh filename=exported_meshes/leg_lower.stl scale=0.001 0.001 0.001

Commit message: fix: improve foot friction and contact geometry for walking
- scene.py: set plane lateralFriction=1.0 explicitly (was default 0.5,
  halving effective friction via geometric mean with foot contact)
- sim_config.yaml: foot_lateral 1.0→3.0 (compensates for point contact
  geometry vs real rubber pad area), foot_spinning 0.3→0.05
- urdf_writer.py: add capsule shape to CollisionPrimitive
- generate_urdf.py: replace link3 sphere with capsule (r=5mm, l=5mm,
  Rx(90deg) oriented along Y for 15mm contact patch matching foot pad)
- Regenerated facehugger.urdf with 4 capsule collisions

All tests pass. URDF loads in PyBullet DIRECT.

File: code/simulation/generated/facehugger.urdf (robot description, URDF)
Before this commit: robot facehugger, 13 links, 12 joints
Links:
- link bl_link3: geometry collision capsule length=0.005 radius=0.005; visual mesh filename=exported_meshes/leg_lower.stl scale=0.001 0.001 0.001
- link br_link3: geometry collision capsule length=0.005 radius=0.005; visual mesh filename=exported_meshes/leg_lower.stl scale=0.001 0.001 0.001
- link fl_link3: geometry collision capsule length=0.005 radius=0.005; visual mesh filename=exported_meshes/leg_lower.stl scale=0.001 0.001 0.001
- link fr_link3: geometry collision capsule length=0.005 radius=0.005; visual mesh filename=exported_meshes/leg_lower.stl scale=0.001 0.001 0.001

Commit message: sim: analytic collision shapes, stable physics, dead code removal (#115) Wiki updates
Likely the last commit before a while because the simulation is stable and the code has been cleaned up.

* feat(blender): add math-space angle display to FH Clips panel

* refactor: rename firmware_port → animation_tools

* refactor: update all firmware_port imports to animation_tools

* fix(.gitignore): scope Lib pattern to repo root to avoid matching animation/lib

* fix: re-export all clips with corrected _LINK1_DELTA_SIGN (+1 for all legs)

* fix: config.h clamp corrections, URDF limits table, remove python port

* docs+test: update firmware_sil README and remove test_clip_player after python port removal

* chore: refresh Fusion export (COM coordinates)

* feat(sim): add positionGain/velocityGain to motor control + sphere foot collision

- Add motor.position_gain (0.5) and motor.velocity_gain (2.0) to sim_config.yaml
- Pass positionGain/velocityGain through all setJointMotorControl2 calls
  (motor.py, sil_bridge.py, ws_sim.py, runner.py)
- Add kp/kd fields to RobotConfig, loaded from sim_config.yaml
- Add sphere collision shapes at each foot tip (radius 15mm) to simulate
  elastic-band grip, constrained via fixed joint to link3
- Add positionGain/velocityGain debug sliders with finalize() output

* chore(sim): bump solver iterations to 300

* fix(sim): disable link3 mesh collision so foot spheres are sole contact

setCollisionFilterGroupMask(robot_id, link_idx, 0, 0) on each link3
link — the mesh convex hull no longer collides with the ground plane.
Only the sphere (zero-mass body constrained at foot tip) makes contact,
eliminating competing collision surfaces that caused instability.

* revert(sim): remove foot sphere collision — unstable at init

The createMultiBody-at-origin then createConstraint snap pattern
caused the constraint solver to jerk spheres from (0,0,0) to the
foot tips on first stepSimulation, transferring explosive impulses
into the leg joints. Joints maxed torque immediately.

Keep positionGain/velocityGain changes — those alone provide the
5x stronger stance tracking needed to resist foot sliding.

* fix(sim): zero link damping + disable default joint motors

Two fixes for sliding-at-rest:
1. Set linearDamping=0, angularDamping=0 on all links (PyBullet defaults
   to 0.04 which creates drag forces during joint motion).
2. Disable loadURDF's built-in joint motor friction by setting
   VELOCITY_CONTROL force=0 on every joint before POSITION_CONTROL.

Added damping.linear/damping.angular to sim_config.yaml.

* feat(sim): add contact force diagnostic to ws_sim (--debug)

RobotSim gains --debug mode with two diagnostics:
1. Startup: prints spawn height + checks whether each foot touches ground
2. Per-frame (every 60 steps / 0.25s): prints per-foot contact points with
   normal force, lateral friction forces, contact normal direction,
   and body base position + orientation.

No physics changes — diagnostic only, for investigating the standing-slide
bug. Pass --debug to ws_sim or python -m firmware_sil.ws_sim --debug.

* fix(sim): spawn at firmware NEUTRAL pose instead of shared STANCE_DEG

Root cause of standing-slide: sim spawned with STANCE_DEG
{hip:-40,knee:-60} for all legs, but firmware NEUTRAL from
neutral_pose.h has per-leg values:
  FR: hip=-60, knee=-37   FL: hip=-60, knee=-40
  BR: hip=-50, knee=-50   BL: hip=-60, knee=-35

On first tick, firmware snapped all 12 joints 10-25 deg,
creating violent impact forces. Sim now starts in the exact
same pose the firmware expects.

_NEUTRAL_HIP_KNEE derived from NEUTRAL[] math-space through
translateToServo(CALIB=90) then servo_angles_to_joint_targets.

* chore: remove dead Python-port code and stale config

- Remove run_gait() from runner.py (gaits.py no longer exists)
- Remove STANCE_DEG from paths.py (unused, superseded by per-leg NEUTRAL)
- Remove --python-port flag handling from facehugger.py and simulate.py
- Remove visual_flip_rpy_deg from config yaml and generate_urdf.py
- Update firmware_sil/__init__.py docstring (no more Python-port counterparts)

All 169 tests pass.

* fix: eliminate manual sync risks, fix stale wiki/docs

- sim_monitor: STALL_TORQUE_NM now syncs from facehugger_config.yaml's
  servo.effort_nm via set_stall_torque(). Called once in
  scene.connect_and_setup(), so changing the yaml shifts all bands.
- sim_config.yaml: remove solver.timestep (always 1/240 Hz, the
  firmware tick rate; single source in pybullet_sim/paths.py).
- firmware_sil/sil_bridge: LEG_ID_TO_URDF_AXIS_SIGN now read from the
  generated URDF at runtime (_build_urdf_axis_signs) instead of the
  old hardcoded dict. The URDF is the kinematic source of truth.
- Update __init__.py and test fixtures to match.
- Wiki/README/CLAUDE.md: remove all --python, gaits.py, verify_export_parity
  references. Update code-location tables and file maps.

All 173 tests pass.

* feat: replace STL collision with analytic primitives on leg links

- urdf_writer.py: add CollisionPrimitive dataclass (sphere/box) and
  collision_override parameter to link(). When override is provided,
  emit analytic geometry instead of STL mesh for collision.
- generate_urdf.py: compute foot tip once in _build_state(), store in
  _GenState. Emit sphere (r=5mm) at foot tip for link3, boxes (15mm
  cross-section) along bone direction for link1 and link2.
- R-pair link3 foot tip applies Ry(pi) mirror via (-x, y, -z) transform
  to match the mesh_rpy flip on the visual.
- base_link keeps STL collision (chassis shape matters for flip/drop).
- Regenerated facehugger.urdf.

All 60 urdf/foot_tip/joint tests pass. URDF loads in PyBullet DIRECT.

* fix: use full 3D rotation for link1/link2 box collision

The old Ry-only approach assumed bones were in the XZ plane, but the
link1 bone (shoulder-to-hip) has a 22.4mm Y component. Now computes
proper Rz(yaw)*Ry(pitch) RPY from the normalized bone vector.

L-pair link1: pitch=0.55rad yaw=2.70rad
R-pair link1: pitch=0.55rad yaw=0.45rad
Link2 bones: essentially XZ-plane (Y=0.2mm) so yaw~0/pi as expected.

* tune: retune sim_config for analytic collision shapes

With sphere foot-tip contact replacing STL mesh collision, the solver
converges faster and needs stiffer contact params:
- contact.stiffness: 30000 -> 80000 (less penetration)
- contact.damping: 100 -> 1000  (absorb oscillation)
- contact.restitution: 0.0 -> 0.1 (slight compliance at feet;
  base_link keeps default 0.0 — only link3 joints get this value)
- friction.foot_lateral: 2.5 -> 1.0 (rubber-on-floor range)
- motor.position_gain: 0.5 -> 1.5 (DSS-230MG is stiff at 30kg.cm)

* fix: correct position_gain — old kp=0.5 was always too aggressive

The jitter reported in float mode is pre-existing, not caused by
collision shape changes. Both old (STL mesh) and new (analytic)
URDFs saturate 8-12/12 joints at kp>=0.3 in float mode.

Root cause: PyBullet POSITION_CONTROL with kp>=0.3 oscillates at
the link inertia without external damping. With kp=0.1, kd=0.5:
- Float mode: 0/12 saturated, 0.000 deg error
- With gravity: 0/12 saturated, max 0.05 deg error, max 0.73 Nm
  (25% of stall — exactly what you want for holding stance)

The original kp=0.5 was already saturating 8/12 joints with gravity.
No collision issue here — just a long-standing gain problem now fixed.

* fix: improve foot friction and contact geometry for walking

- scene.py: set plane lateralFriction=1.0 explicitly (was default 0.5,
  halving effective friction via geometric mean with foot contact)
- sim_config.yaml: foot_lateral 1.0→3.0 (compensates for point contact
  geometry vs real rubber pad area), foot_spinning 0.3→0.05
- urdf_writer.py: add capsule shape to CollisionPrimitive
- generate_urdf.py: replace link3 sphere with capsule (r=5mm, l=5mm,
  Rx(90deg) oriented along Y for 15mm contact patch matching foot pad)
- Regenerated facehugger.urdf with 4 capsule collisions

All tests pass. URDF loads in PyBullet DIRECT.

* tune: settle on stable sim_config — moderate contact, zero restitution

After iteration: stiffness=20000 (prevents jitter from over-stiff contact),
damping=500 (absorbs oscillation without slowing solver), restitution=0.0
(inelastic — robot has no rubber bounce in real life). These values produce
stable stance with the analytic collision shapes.

* docs: add simulation limitations section to wiki

Captures known gaps: contact model (capsule vs rubber pads), body dynamics
(light chassis relative to leg servos causes bounciness), and self-collision
simplifications. The sim is authoritative for servo-level joint motion, not
full-body dynamics.

* chore: update animation exports and rigged blend file

File: code/simulation/generated/facehugger.urdf (robot description, URDF)
Before this commit: robot facehugger, 13 links, 12 joints
Links:
- link bl_link1: geometry collision box size=0.060840 0.015000 0.015000; visual mesh filename=exported_meshes/leg_shoulder_R.stl scale=0.001 0.001 0.001
- link bl_link2: geometry collision box size=0.074700 0.015000 0.015000; visual mesh filename=exported_meshes/leg_upper.stl scale=0.001 0.001 0.001
- link bl_link3: geometry collision capsule length=0.005 radius=0.005; visual mesh filename=exported_meshes/leg_lower.stl scale=0.001 0.001 0.001
- link br_link1: geometry collision box size=0.060840 0.015000 0.015000; visual mesh filename=exported_meshes/leg_shoulder_L.stl scale=0.001 0.001 0.001
- link br_link2: geometry collision box size=0.074700 0.015000 0.015000; visual mesh filename=exported_meshes/leg_upper.stl scale=0.001 0.001 0.001
- link br_link3: geometry collision capsule length=0.005 radius=0.005; visual mesh filename=exported_meshes/leg_lower.stl scale=0.001 0.001 0.001
- link fl_link1: geometry collision box size=0.060840 0.015000 0.015000; visual mesh filename=exported_meshes/leg_shoulder_L.stl scale=0.001 0.001 0.001
- link fl_link2: geometry collision box size=0.074700 0.015000 0.015000; visual mesh filename=exported_meshes/leg_upper.stl scale=0.001 0.001 0.001
- link fl_link3: geometry collision capsule length=0.005 radius=0.005; visual mesh filename=exported_meshes/leg_lower.stl scale=0.001 0.001 0.001
- link fr_link1: geometry collision box size=0.060840 0.015000 0.015000; visual mesh filename=exported_meshes/leg_shoulder_R.stl scale=0.001 0.001 0.001
- link fr_link2: geometry collision box size=0.074700 0.015000 0.015000; visual mesh filename=exported_meshes/leg_upper.stl scale=0.001 0.001 0.001
- link fr_link3: geometry collision capsule length=0.005 radius=0.005; visual mesh filename=exported_meshes/leg_lower.stl scale=0.001 0.001 0.001
